File: druid/xmobile_audio.sch (KiCad schematic (older format))
At the start: 28 parts, among them P4 CONN_MICROPHONE, P5 CONN_MICROPHONE

Commit message: - Переделана клавиатура - установлены все корпуса микросхем
Parts:
- C10, C11, C12, C13, C14, C15, C16, C17, C18, C19, C20, C21, C4, C5, C6, C7, C8, C9: footprint (none) -> Capacitors_SMD:C_1206_HandSoldering; symbol C -> C-RESCUE-xmobile
- D2, D3, D4, D5, D6, D7, D8, D9: footprint (none) -> LEDs:LED_0603; symbol LED -> LED-RESCUE-xmobile
- P4, P5: footprint (none) -> Connectors_Molex:Molex_KK-6410-02_02x2.54mm_Straight
Connections:
- wire segments 68 -> 40

Commit message: Переместил посадочные места по кучкам
Parts:
- P4: footprint Connectors_Molex:Molex_KK-6410-02_02x2.54mm_Straight -> Connectors_Hirose:Hirose_DF13-02P-1.25DSA_02x1.25mm_Straight
Changed lines of the file:
@@
 F 0 "P4" V 7575 2425 40  0000 C CNN
 F 1 "CONN_MICROPHONE" V 7775 2425 40  0000 C CNN
-F 2 "Connectors_Molex:Molex_KK-6410-02_02x2.54mm_Straight" H 7625 2425 60  0001 C CNN
+F 2 "Connectors_Hirose:Hirose_DF13-02P-1.25DSA_02x1.25mm_Straight" H 7625 2425 60  0001 C CNN
 F 3 "" H 7625 2425 60  0001 C CNN
 	1    7625 2425

Commit message: Заменил посадочные места для некоторых контактных расчёсок
Parts:
- P5: footprint Connectors_Molex:Molex_KK-6410-02_02x2.54mm_Straight -> Connectors_JAE:JAE_LY20-08P-2T_2x04x2.00mm_Straight
Changed lines of the file:
@@
 F 0 "P5" V 7825 4975 40  0000 C CNN
 F 1 "CONN_MICROPHONE" V 8025 4975 40  0000 C CNN
-F 2 "Connectors_Molex:Molex_KK-6410-02_02x2.54mm_Straight" H 7875 4975 60  0001 C CNN
+F 2 "Connectors_JAE:JAE_LY20-08P-2T_2x04x2.00mm_Straight" H 7875 4975 60  0001 C CNN
 F 3 "" H 7875 4975 60  0001 C CNN
 	1    7875 4975

Commit message: Соединеты проводникаи отдельные блоки и начато подключение SIM800 к XMEGA
Parts:
- P4: footprint Connectors_Hirose:Hirose_DF13-02P-1.25DSA_02x1.25mm_Straight -> Connectors_JAE:JAE_LY20-04P-2T_2x02x2.00mm_Straight
- P5: footprint Connectors_JAE:JAE_LY20-08P-2T_2x04x2.00mm_Straight -> Connectors_JAE:JAE_LY20-04P-2T_2x02x2.00mm_Straight
Changed lines of the file:
@@
 F 0 "P4" V 7575 2425 40  0000 C CNN
 F 1 "CONN_MICROPHONE" V 7775 2425 40  0000 C CNN
-F 2 "Connectors_Hirose:Hirose_DF13-02P-1.25DSA_02x1.25mm_Straight" H 7625 2425 60  0001 C CNN
+F 2 "Connectors_JAE:JAE_LY20-04P-2T_2x02x2.00mm_Straight" H 7625 2425 60  0001 C CNN
 F 3 "" H 7625 2425 60  0001 C CNN
 	1    7625 2425
@@
 F 0 "P5" V 7825 4975 40  0000 C CNN
 F 1 "CONN_MICROPHONE" V 8025 4975 40  0000 C CNN
-F 2 "Connectors_JAE:JAE_LY20-08P-2T_2x04x2.00mm_Straight" H 7875 4975 60  0001 C CNN
+F 2 "Connectors_JAE:JAE_LY20-04P-2T_2x02x2.00mm_Straight" H 7875 4975 60  0001 C CNN
 F 3 "" H 7875 4975 60  0001 C CNN
 	1    7875 4975
