File: druid/xmobile_audio.sch (KiCad schematic (older format))
At the start: 28 parts, among them P4 CONN_MICROPHONE, P5 CONN_MICROPHONE

Commit message: Old buttons replaced by membran buttons (electic and pcb) Added pcb for MAX7370 Cleared PCBs of resistor, capacitors and diodes
Parts:
- C10, C11, C12, C13, C14, C15, C16, C17, C18, C19, C20, C21, C4, C5, C6, C7, C8, C9: footprint Capacitors_SMD:C_1206_HandSoldering -> (none)
- D2, D3, D4, D5, D6, D7, D8, D9: footprint LEDs:LED_0603 -> (none)
Connections:
- wire segments 40 -> 41
Changed lines of the file:
@@
 F 0 "C10" H 5650 2050 40  0000 L CNN
 F 1 "10pF" H 5656 1865 40  0000 L CNN
-F 2 "Capacitors_SMD:C_1206_HandSoldering" H 5688 1800 30  0000 C CNN
+F 2 "" H 5688 1800 30  0000 C CNN
 F 3 "" H 5650 1950 60  0000 C CNN
 	1    5650 1950
@@
 F 0 "C16" H 6150 2050 40  0000 L CNN
 F 1 "33pF" H 6156 1865 40  0000 L CNN
-F 2 "Capacitors_SMD:C_1206_HandSoldering" H 6188 1800 30  0000 C CNN
+F 2 "" H 6188 1800 30  0000 C CNN
 F 3 "" H 6150 1950 60  0000 C CNN
 	1    6150 1950
@@
 F 0 "C11" H 5650 2550 40  0000 L CNN
 F 1 "10pF" H 5656 2365 40  0000 L CNN
-F 2 "Capacitors_SMD:C_1206_HandSoldering" H 5688 2300 30  0000 C CNN
+F 2 "" H 5688 2300 30  0000 C CNN
 F 3 "" H 5650 2450 60  0000 C CNN
 	1    5650 2450
@@
 F 0 "C17" H 6150 2550 40  0000 L CNN
 F 1 "33pF" H 6156 2365 40  0000 L CNN
-F 2 "Capacitors_SMD:C_1206_HandSoldering" H 6188 2300 30  0000 C CNN
+F 2 "" H 6188 2300 30  0000 C CNN
 F 3 "" H 6150 2450 60  0000 C CNN
 	1    6150 2450
@@
 F 0 "C18" H 6150 3050 40  0000 L CNN
 F 1 "33pF" H 6156 2865 40  0000 L CNN
-F 2 "Capacitors_SMD:C_1206_HandSoldering" H 6188 2800 30  0000 C CNN
+F 2 "" H 6188 2800 30  0000 C CNN
 F 3 "" H 6150 2950 60  0000 C CNN
 	1    6150 2950
@@
 F 0 "C12" H 5650 3050 40  0000 L CNN
 F 1 "10pF" H 5656 2865 40  0000 L CNN
-F 2 "Capacitors_SMD:C_1206_HandSoldering" H 5688 2800 30  0000 C CNN
+F 2 "" H 5688 2800 30  0000 C CNN
 F 3 "" H 5650 2950 60  0000 C CNN
 	1    5650 2950
@@
 F 0 "D6" H 7100 2000 50  0000 C CNN
 F 1 "LED BLUE" H 7100 1800 50  0000 C CNN
-F 2 "LEDs:LED_0603" H 7100 1900 60  0000 C CNN
+F 2 "" H 7100 1900 60  0000 C CNN
 F 3 "" H 7100 1900 60  0000 C CNN
 	1    7100 1900
@@
 F 0 "D2" H 6725 2000 50  0000 C CNN
 F 1 "LED BLUE" H 6725 1800 50  0000 C CNN
-F 2 "LEDs:LED_0603" H 6725 1900 60  0000 C CNN
+F 2 "" H 6725 1900 60  0000 C CNN
 F 3 "" H 6725 1900 60  0000 C CNN
 	1    6725 1900
@@
 F 0 "D7" H 7100 3100 50  0000 C CNN
 F 1 "LED BLUE" H 7100 2900 50  0000 C CNN
-F 2 "LEDs:LED_0603" H 7100 3000 60  0000 C CNN
+F 2 "" H 7100 3000 60  0000 C CNN
 F 3 "" H 7100 3000 60  0000 C CNN
 	1    7100 3000
@@
 F 0 "D3" H 6725 3100 50  0000 C CNN
 F 1 "LED BLUE" H 6725 2900 50  0000 C CNN
-F 2 "LEDs:LED_0603" H 6725 3000 60  0000 C CNN
+F 2 "" H 6725 3000 60  0000 C CNN
 F 3 "" H 6725 3000 60  0000 C CNN
 	1    6725 3000
@@
 	6150 2150 6150 2250
 Wire Wire Line
-	6725 1700 6725 1600
+	6725 1600 6725 1750
 Wire Wire Line
 	6725 1600 7100 1600
 Wire Wire Line
-	7100 1600 7100 1700
-Wire Wire Line
-	6725 2200 6725 2100
+	7100 1600 7100 1750
+Wire Wire Line
+	6725 2050 6725 2200
 Wire Wire Line
 	5650 2200 7100 2200
 Wire Wire Line
-	7100 2100 7100 2325
-Wire Wire Line
-	6725 2700 6725 2800
+	7100 2050 7100 2325
+Wire Wire Line
+	6725 2700 6725 2850
 Wire Wire Line
 	5650 2700 7100 2700
@@
 	7100 2525 7100 2800
 Wire Wire Line
-	6725 3200 6725 3300
+	6725 3150 6725 3300
 Wire Wire Line
 	6725 3300 7100 3300
 Wire Wire Line
-	7100 3300 7100 3200
+	7100 3300 7100 3150
 Connection ~ 6150 2200
 Connection ~ 5650 2200
@@
 F 0 "C4" H 4025 4600 40  0000 L CNN
 F 1 "10pF" H 4031 4415 40  0000 L CNN
-F 2 "Capacitors_SMD:C_1206_HandSoldering" H 4063 4350 30  0000 C CNN
+F 2 "" H 4063 4350 30  0000 C CNN
 F 3 "" H 4025 4500 60  0000 C CNN
 	1    4025 4500
@@
 F 0 "C7" H 4525 4600 40  0000 L CNN
 F 1 "33pF" H 4531 4415 40  0000 L CNN
-F 2 "Capacitors_SMD:C_1206_HandSoldering" H 4563 4350 30  0000 C CNN
+F 2 "" H 4563 4350 30  0000 C CNN
 F 3 "" H 4525 4500 60  0000 C CNN
 	1    4525 4500
@@
 F 0 "C5" H 4025 5100 40  0000 L CNN
 F 1 "10pF" H 4031 4915 40  0000 L CNN
-F 2 "Capacitors_SMD:C_1206_HandSoldering" H 4063 4850 30  0000 C CNN
+F 2 "" H 4063 4850 30  0000 C CNN
 F 3 "" H 4025 5000 60  0000 C CNN
 	1    4025 5000
@@
 F 0 "C8" H 4525 5100 40  0000 L CNN
 F 1 "33pF" H 4531 4915 40  0000 L CNN
-F 2 "Capacitors_SMD:C_1206_HandSoldering" H 4563 4850 30  0000 C CNN
+F 2 "" H 4563 4850 30  0000 C CNN
 F 3 "" H 4525 5000 60  0000 C CNN
 	1    4525 5000
@@
 F 0 "C9" H 4525 5600 40  0000 L CNN
 F 1 "33pF" H 4531 5415 40  0000 L CNN
-F 2 "Capacitors_SMD:C_1206_HandSoldering" H 4563 5350 30  0000 C CNN
+F 2 "" H 4563 5350 30  0000 C CNN
 F 3 "" H 4525 5500 60  0000 C CNN
 	1    4525 5500
@@
 F 0 "C6" H 4025 5600 40  0000 L CNN
 F 1 "10pF" H 4031 5415 40  0000 L CNN
-F 2 "Capacitors_SMD:C_1206_HandSoldering" H 4063 5350 30  0000 C CNN
+F 2 "" H 4063 5350 30  0000 C CNN
 F 3 "" H 4025 5500 60  0000 C CNN
 	1    4025 5500
@@
 F 0 "C13" H 5900 4600 40  0000 L CNN
 F 1 "10pF" H 5906 4415 40  0000 L CNN
-F 2 "Capacitors_SMD:C_1206_HandSoldering" H 5938 4350 30  0000 C CNN
+F 2 "" H 5938 4350 30  0000 C CNN
 F 3 "" H 5900 4500 60  0000 C CNN
 	1    5900 4500
@@
 F 0 "C19" H 6400 4600 40  0000 L CNN
 F 1 "33pF" H 6406 4415 40  0000 L CNN
-F 2 "Capacitors_SMD:C_1206_HandSoldering" H 6438 4350 30  0000 C CNN
+F 2 "" H 6438 4350 30  0000 C CNN
 F 3 "" H 6400 4500 60  0000 C CNN
 	1    6400 4500
@@
 F 0 "C14" H 5900 5100 40  0000 L CNN
 F 1 "10pF" H 5906 4915 40  0000 L CNN
-F 2 "Capacitors_SMD:C_1206_HandSoldering" H 5938 4850 30  0000 C CNN
+F 2 "" H 5938 4850 30  0000 C CNN
 F 3 "" H 5900 5000 60  0000 C CNN
 	1    5900 5000
@@
 F 0 "C20" H 6400 5100 40  0000 L CNN
 F 1 "33pF" H 6406 4915 40  0000 L CNN
-F 2 "Capacitors_SMD:C_1206_HandSoldering" H 6438 4850 30  0000 C CNN
+F 2 "" H 6438 4850 30  0000 C CNN
 F 3 "" H 6400 5000 60  0000 C CNN
 	1    6400 5000
@@
 F 0 "C21" H 6400 5600 40  0000 L CNN
 F 1 "33pF" H 6406 5415 40  0000 L CNN
-F 2 "Capacitors_SMD:C_1206_HandSoldering" H 6438 5350 30  0000 C CNN
+F 2 "" H 6438 5350 30  0000 C CNN
 F 3 "" H 6400 5500 60  0000 C CNN
 	1    6400 5500
@@
 F 0 "C15" H 5900 5600 40  0000 L CNN
 F 1 "10pF" H 5906 5415 40  0000 L CNN
-F 2 "Capacitors_SMD:C_1206_HandSoldering" H 5938 5350 30  0000 C CNN
+F 2 "" H 5938 5350 30  0000 C CNN
 F 3 "" H 5900 5500 60  0000 C CNN
 	1    5900 5500
@@
 F 0 "D8" H 7350 4550 50  0000 C CNN
 F 1 "LED BLUE" H 7350 4350 50  0000 C CNN
-F 2 "LEDs:LED_0603" H 7350 4450 60  0000 C CNN
+F 2 "" H 7350 4450 60  0000 C CNN
 F 3 "" H 7350 4450 60  0000 C CNN
 	1    7350 4450
@@
 F 0 "D4" H 6975 4550 50  0000 C CNN
 F 1 "LED BLUE" H 6975 4350 50  0000 C CNN
-F 2 "LEDs:LED_0603" H 6975 4450 60  0000 C CNN
+F 2 "" H 6975 4450 60  0000 C CNN
 F 3 "" H 6975 4450 60  0000 C CNN
 	1    6975 4450
@@
 F 0 "D9" H 7350 5650 50  0000 C CNN
 F 1 "LED BLUE" H 7350 5450 50  0000 C CNN
-F 2 "LEDs:LED_0603" H 7350 5550 60  0000 C CNN
+F 2 "" H 7350 5550 60  0000 C CNN
 F 3 "" H 7350 5550 60  0000 C CNN
 	1    7350 5550
@@
 F 0 "D5" H 6975 5650 50  0000 C CNN
 F 1 "LED BLUE" H 6975 5450 50  0000 C CNN
-F 2 "LEDs:LED_0603" H 6975 5550 60  0000 C CNN
+F 2 "" H 6975 5550 60  0000 C CNN
 F 3 "" H 6975 5550 60  0000 C CNN
 	1    6975 5550
@@
 	6400 4700 6400 4800
 Wire Wire Line
-	6975 4250 6975 4150
+	6975 4150 6975 4300
 Wire Wire Line
 	6975 4150 7350 4150
 Wire Wire Line
-	7350 4150 7350 4250
-Wire Wire Line
-	6975 4750 6975 4650
+	7350 4150 7350 4300
+Wire Wire Line
+	6975 4600 6975 4750
 Wire Wire Line
 	4025 4750 7350 4750
 Wire Wire Line
-	7350 4650 7350 4875
-Wire Wire Line
-	6975 5250 6975 5350
+	7350 4600 7350 4875
+Wire Wire Line
+	6975 5250 6975 5400
 Wire Wire Line
 	4025 5250 7350 5250
 Wire Wire Line
-	7350 5075 7350 5350
-Wire Wire Line
-	6975 5750 6975 5850
+	7350 5075 7350 5400
+Wire Wire Line
+	6975 5700 6975 5850
 Wire Wire Line
 	6975 5850 7350 5850
 Wire Wire Line
-	7350 5850 7350 5750
+	7350 5850 7350 5700
 Connection ~ 6400 4750
 Connection ~ 5900 4750
@@
 Text HLabel 4025 5250 0    60   Input ~ 0
 AUDIO_SPKN
+Wire Wire Line
+	7100 2825 7100 2850
 $EndSCHEMATC

Commit message: Add some packages
Parts:
- removed C11, C12, C13, C14, C15, C4, C5, C6: 10pF, symbol C-RESCUE-xmobile
- removed C17, C18, C19, C20, C21, C7, C8, C9: 33pF, symbol C-RESCUE-xmobile
- removed P4, P5: CONN_MICROPHONE, Connectors_JAE:JAE_LY20-04P-2T_2x02x2.00mm_Straight, symbol CONN_2
- added C? (x8): 10pF, Capacitors_SMD:C_0402, symbol C-RESCUE-xmobile
- added C? (x8): 33pF, Capacitors_SMD:C_0402, symbol C-RESCUE-xmobile
- added W?: MIC, Measurement_Points:Test_Point_2Pads, symbol TEST
- added W?: SPK, Measurement_Points:Test_Point_2Pads, symbol TEST
- C10: footprint (none) -> Capacitors_SMD:C_0402; case (none) -> 0402 In; example (none) -> https://eu.mouser.com/ProductDetail/AVX/04026A100JAT2A?qs=s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
- C16: footprint (none) -> Capacitors_SMD:C_0402; case (none) -> 0402 In; example (none) -> https://eu.mouser.com/ProductDetail/KEMET/C0402C330J9RACAUT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
Connections:
- wire segments 41 -> 40

Commit message: Add packages for LEDs
Parts:
- removed D3, D4, D5, D6, D7, D8, D9: LED BLUE, symbol LED-RESCUE-xmobile
- added D? (x7): LED BLUE, LEDs:LED_0402, symbol LED-RESCUE-xmobile
- D2: footprint (none) -> LEDs:LED_0402; case (none) -> 0402 In; example (none) -> https://ru.mouser.com/ProductDetail/ROHM-Semiconductor/SMLP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
- W? (x2): symbol TEST -> TEST-RESCUE-xmobile; case (none) -> 2 pads
Changed lines of the file:
@@
 GND
-$Comp
-L LED-RESCUE-xmobile D6
-U 1 1 5A9F1A37
-P 7100 1900
-F 0 "D6" H 7100 2000 50  0000 C CNN
-F 1 "LED BLUE" H 7100 1800 50  0000 C CNN
-F 2 "" H 7100 1900 60  0000 C CNN
-F 3 "" H 7100 1900 60  0000 C CNN
-	1    7100 1900
-	0    1    1    0
-$EndComp
 $Comp
 L LED-RESCUE-xmobile D2
@@
 F 0 "D2" H 6725 2000 50  0000 C CNN
 F 1 "LED BLUE" H 6725 1800 50  0000 C CNN
-F 2 "" H 6725 1900 60  0000 C CNN
-F 3 "" H 6725 1900 60  0000 C CNN
+F 2 "LEDs:LED_0402" H 6725 1900 60  0001 C CNN
+F 3 "https://ru.mouser.com/datasheet/2/348/sml-p1-e-1139198.pdf" H 6725 1900 60  0001 C CNN
+F 4 "https://ru.mouser.com/ProductDetail/ROHM-Semiconductor/SMLP13BC8TT86?qs=sGAEpiMZZMuCm2JlHBGefhkTP7nu0Fg7%2fyfWOmjl5dYVsL3Njh32dw%3d%3d" H 6725 1900 60  0001 C CNN "example"
+F 5 "0402 In" H 6575 2000 30  0000 C CNN "case"
 	1    6725 1900
-	0    -1   -1   0
-$EndComp
-$Comp
-L LED-RESCUE-xmobile D7
-U 1 1 5A9F1A45
-P 7100 3000
-F 0 "D7" H 7100 3100 50  0000 C CNN
-F 1 "LED BLUE" H 7100 2900 50  0000 C CNN
-F 2 "" H 7100 3000 60  0000 C CNN
-F 3 "" H 7100 3000 60  0000 C CNN
-	1    7100 3000
-	0    1    1    0
-$EndComp
-$Comp
-L LED-RESCUE-xmobile D3
-U 1 1 5A9F1A4C
-P 6725 3000
-F 0 "D3" H 6725 3100 50  0000 C CNN
-F 1 "LED BLUE" H 6725 2900 50  0000 C CNN
-F 2 "" H 6725 3000 60  0000 C CNN
-F 3 "" H 6725 3000 60  0000 C CNN
-	1    6725 3000
 	0    -1   -1   0
 $EndComp
@@
 Text Label 5900 4300 1    60   ~ 0
 GND
-$Comp
-L LED-RESCUE-xmobile D8
-U 1 1 5A9F1ADC
-P 7350 4450
-F 0 "D8" H 7350 4550 50  0000 C CNN
-F 1 "LED BLUE" H 7350 4350 50  0000 C CNN
-F 2 "" H 7350 4450 60  0000 C CNN
-F 3 "" H 7350 4450 60  0000 C CNN
-	1    7350 4450
-	0    1    1    0
-$EndComp
-$Comp
-L LED-RESCUE-xmobile D4
-U 1 1 5A9F1AE3
-P 6975 4450
-F 0 "D4" H 6975 4550 50  0000 C CNN
-F 1 "LED BLUE" H 6975 4350 50  0000 C CNN
-F 2 "" H 6975 4450 60  0000 C CNN
-F 3 "" H 6975 4450 60  0000 C CNN
-	1    6975 4450
-	0    -1   -1   0
-$EndComp
-$Comp
-L LED-RESCUE-xmobile D9
-U 1 1 5A9F1AEA
-P 7350 5550
-F 0 "D9" H 7350 5650 50  0000 C CNN
-F 1 "LED BLUE" H 7350 5450 50  0000 C CNN
-F 2 "" H 7350 5550 60  0000 C CNN
-F 3 "" H 7350 5550 60  0000 C CNN
-	1    7350 5550
-	0    1    1    0
-$EndComp
-$Comp
-L LED-RESCUE-xmobile D5
-U 1 1 5A9F1AF1
-P 6975 5550
-F 0 "D5" H 6975 5650 50  0000 C CNN
-F 1 "LED BLUE" H 6975 5450 50  0000 C CNN
-F 2 "" H 6975 5550 60  0000 C CNN
-F 3 "" H 6975 5550 60  0000 C CNN
-	1    6975 5550
-	0    -1   -1   0
-$EndComp
 Wire Wire Line
 	4025 4700 4025 4800
@@
 	7100 2700 7100 2850
 $Comp
-L TEST W?
+L TEST-RESCUE-xmobile W?
 U 1 1 5C6D0927
 P 7500 2450
+AR Path="/5C6D0927" Ref="W?"  Part="1"
+AR Path="/5A9ED5F5/5C6D0927" Ref="W?"  Part="1"
 F 0 "W?" H 7500 2510 50  0000 C CNN
 F 1 "MIC" H 7500 2380 50  0000 C CNN
-F 2 "Measurement_Points:Test_Point_2Pads" H 7450 2600 50  0000 C CNN
+F 2 "Measurement_Points:Test_Point_2Pads" H 7450 2600 50  0001 C CNN
 F 3 "" H 7500 2450 50  0000 C CNN
+F 4 "2 pads" H 7500 2550 30  0000 C CNN "case"
 	1    7500 2450
 	0    1    1    0
@@
 	7500 2200 7500 2250
 $Comp
-L TEST W?
+L TEST-RESCUE-xmobile W?
 U 1 1 5C6D0EE0
 P 7650 5000
+AR Path="/5C6D0EE0" Ref="W?"  Part="1"
+AR Path="/5A9ED5F5/5C6D0EE0" Ref="W?"  Part="1"
 F 0 "W?" H 7650 5060 50  0000 C CNN
 F 1 "SPK" H 7650 4930 50  0000 C CNN
-F 2 "Measurement_Points:Test_Point_2Pads" H 7600 5150 50  0000 C CNN
+F 2 "Measurement_Points:Test_Point_2Pads" H 7600 5150 50  0001 C CNN
 F 3 "" H 7650 5000 50  0000 C CNN
+F 4 "2 pads" H 7650 5100 30  0000 C CNN "case"
 	1    7650 5000
 	0    1    1    0
@@
 	1    0    0    -1
 $EndComp
+$Comp
+L LED-RESCUE-xmobile D?
+U 1 1 5C6C7622
+P 7100 1900
+F 0 "D?" H 7100 2000 50  0000 C CNN
+F 1 "LED BLUE" H 7100 1800 50  0000 C CNN
+F 2 "LEDs:LED_0402" H 7100 1900 60  0001 C CNN
+F 3 "https://ru.mouser.com/datasheet/2/348/sml-p1-e-1139198.pdf" H 7100 1900 60  0001 C CNN
+F 4 "https://ru.mouser.com/ProductDetail/ROHM-Semiconductor/SMLP13BC8TT86?qs=sGAEpiMZZMuCm2JlHBGefhkTP7nu0Fg7%2fyfWOmjl5dYVsL3Njh32dw%3d%3d" H 7100 1900 60  0001 C CNN "example"
+F 5 "0402 In" H 6950 2000 30  0000 C CNN "case"
+	1    7100 1900
+	0    1    1    0
+$EndComp
+$Comp
+L LED-RESCUE-xmobile D?
+U 1 1 5C6C77F4
+P 7100 3000
+F 0 "D?" H 7100 3100 50  0000 C CNN
+F 1 "LED BLUE" H 7100 2900 50  0000 C CNN
+F 2 "LEDs:LED_0402" H 7100 3000 60  0001 C CNN
+F 3 "https://ru.mouser.com/datasheet/2/348/sml-p1-e-1139198.pdf" H 7100 3000 60  0001 C CNN
+F 4 "https://ru.mouser.com/ProductDetail/ROHM-Semiconductor/SMLP13BC8TT86?qs=sGAEpiMZZMuCm2JlHBGefhkTP7nu0Fg7%2fyfWOmjl5dYVsL3Njh32dw%3d%3d" H 7100 3000 60  0001 C CNN "example"
+F 5 "0402 In" H 6950 3100 30  0000 C CNN "case"
+	1    7100 3000
+	0    1    1    0
+$EndComp
+$Comp
+L LED-RESCUE-xmobile D?
+U 1 1 5C6C796F
+P 6725 3000
+F 0 "D?" H 6725 3100 50  0000 C CNN
+F 1 "LED BLUE" H 6725 2900 50  0000 C CNN
+F 2 "LEDs:LED_0402" H 6725 3000 60  0001 C CNN
+F 3 "https://ru.mouser.com/datasheet/2/348/sml-p1-e-1139198.pdf" H 6725 3000 60  0001 C CNN
+F 4 "https://ru.mouser.com/ProductDetail/ROHM-Semiconductor/SMLP13BC8TT86?qs=sGAEpiMZZMuCm2JlHBGefhkTP7nu0Fg7%2fyfWOmjl5dYVsL3Njh32dw%3d%3d" H 6725 3000 60  0001 C CNN "example"
+F 5 "0402 In" H 6575 3100 30  0000 C CNN "case"
+	1    6725 3000
+	0    -1   -1   0
+$EndComp
+$Comp
+L LED-RESCUE-xmobile D?
+U 1 1 5C6C7BA9
+P 6975 4450
+F 0 "D?" H 6975 4550 50  0000 C CNN
+F 1 "LED BLUE" H 6975 4350 50  0000 C CNN
+F 2 "LEDs:LED_0402" H 6975 4450 60  0001 C CNN
+F 3 "https://ru.mouser.com/datasheet/2/348/sml-p1-e-1139198.pdf" H 6975 4450 60  0001 C CNN
+F 4 "https://ru.mouser.com/ProductDetail/ROHM-Semiconductor/SMLP13BC8TT86?qs=sGAEpiMZZMuCm2JlHBGefhkTP7nu0Fg7%2fyfWOmjl5dYVsL3Njh32dw%3d%3d" H 6975 4450 60  0001 C CNN "example"
+F 5 "0402 In" H 6825 4550 30  0000 C CNN "case"
+	1    6975 4450
+	0    -1   -1   0
+$EndComp
+$Comp
+L LED-RESCUE-xmobile D?
+U 1 1 5C6C7D73
+P 7350 4450
+F 0 "D?" H 7350 4550 50  0000 C CNN
+F 1 "LED BLUE" H 7350 4350 50  0000 C CNN
+F 2 "LEDs:LED_0402" H 7350 4450 60  0001 C CNN
+F 3 "https://ru.mouser.com/datasheet/2/348/sml-p1-e-1139198.pdf" H 7350 4450 60  0001 C CNN
+F 4 "https://ru.mouser.com/ProductDetail/ROHM-Semiconductor/SMLP13BC8TT86?qs=sGAEpiMZZMuCm2JlHBGefhkTP7nu0Fg7%2fyfWOmjl5dYVsL3Njh32dw%3d%3d" H 7350 4450 60  0001 C CNN "example"
+F 5 "0402 In" H 7200 4550 30  0000 C CNN "case"
+	1    7350 4450
+	0    1    1    0
+$EndComp
+$Comp
+L LED-RESCUE-xmobile D?
+U 1 1 5C6C7FDB
+P 7350 5550
+F 0 "D?" H 7350 5650 50  0000 C CNN
+F 1 "LED BLUE" H 7350 5450 50  0000 C CNN
+F 2 "LEDs:LED_0402" H 7350 5550 60  0001 C CNN
+F 3 "https://ru.mouser.com/datasheet/2/348/sml-p1-e-1139198.pdf" H 7350 5550 60  0001 C CNN
+F 4 "https://ru.mouser.com/ProductDetail/ROHM-Semiconductor/SMLP13BC8TT86?qs=sGAEpiMZZMuCm2JlHBGefhkTP7nu0Fg7%2fyfWOmjl5dYVsL3Njh32dw%3d%3d" H 7350 5550 60  0001 C CNN "example"
+F 5 "0402 In" H 7200 5650 30  0000 C CNN "case"
+	1    7350 5550
+	0    1    1    0
+$EndComp
+$Comp
+L LED-RESCUE-xmobile D?
+U 1 1 5C6C809E
+P 6975 5550
+F 0 "D?" H 6975 5650 50  0000 C CNN
+F 1 "LED BLUE" H 6975 5450 50  0000 C CNN
+F 2 "LEDs:LED_0402" H 6975 5550 60  0001 C CNN
+F 3 "https://ru.mouser.com/datasheet/2/348/sml-p1-e-1139198.pdf" H 6975 5550 60  0001 C CNN
+F 4 "https://ru.mouser.com/ProductDetail/ROHM-Semiconductor/SMLP13BC8TT86?qs=sGAEpiMZZMuCm2JlHBGefhkTP7nu0Fg7%2fyfWOmjl5dYVsL3Njh32dw%3d%3d" H 6975 5550 60  0001 C CNN "example"
+F 5 "0402 In" H 6825 5650 30  0000 C CNN "case"
+	1    6975 5550
+	0    -1   -1   0
+$EndComp
 $EndSCHEMATC

Commit message: move to kicad 5
Parts:
- C10, C16, C? (x16): symbol C-RESCUE-xmobile -> xmobile-rescue:C-RESCUE-xmobile
- D2, D? (x7): symbol LED-RESCUE-xmobile -> xmobile-rescue:LED-RESCUE-xmobile
- W? (x2): symbol TEST-RESCUE-xmobile -> xmobile-rescue:TEST-RESCUE-xmobile
Changed lines of the file:
@@
-EESchema Schematic File Version 2
-LIBS:xmobile-rescue
-LIBS:power
-LIBS:device
-LIBS:transistors
-LIBS:conn
-LIBS:linear
-LIBS:regul
-LIBS:74xx
-LIBS:cmos4000
-LIBS:adc-dac
-LIBS:memory
-LIBS:xilinx
-LIBS:microcontrollers
-LIBS:dsp
-LIBS:microchip
-LIBS:analog_switches
-LIBS:motorola
-LIBS:texas
-LIBS:intel
-LIBS:audio
-LIBS:interface
-LIBS:digital-audio
-LIBS:philips
-LIBS:display
-LIBS:cypress
-LIBS:siliconi
-LIBS:opto
-LIBS:atmel
-LIBS:contrib
-LIBS:valves
-LIBS:XC6206P332MR
-LIBS:STF202-22T1G
-LIBS:MCP73871
-LIBS:switch1
-LIBS:SRAM
-LIBS:xmega128a1u_bga100
-LIBS:sim-holders
-LIBS:max7370
-LIBS:tp4056
+EESchema Schematic File Version 4
 LIBS:xmobile-cache
-EELAYER 25 0
+EELAYER 26 0
 EELAYER END
 $Descr A4 11693 8268
@@
 $EndDescr
 $Comp
-L C-RESCUE-xmobile C10
+L xmobile-rescue:C-RESCUE-xmobile C10
 U 1 1 5A9F1A09
 P 5650 1950
@@
 $EndComp
 $Comp
-L C-RESCUE-xmobile C16
+L xmobile-rescue:C-RESCUE-xmobile C16
 U 1 1 5A9F1A10
 P 6150 1950
@@
 GND
 $Comp
-L LED-RESCUE-xmobile D2
+L xmobile-rescue:LED-RESCUE-xmobile D2
 U 1 1 5A9F1A3E
 P 6725 1900
@@
 	7100 2700 7100 2850
 $Comp
-L TEST-RESCUE-xmobile W?
+L xmobile-rescue:TEST-RESCUE-xmobile W?
 U 1 1 5C6D0927
 P 7500 2450
@@
 	7500 2200 7500 2250
 $Comp
-L TEST-RESCUE-xmobile W?
+L xmobile-rescue:TEST-RESCUE-xmobile W?
 U 1 1 5C6D0EE0
 P 7650 5000
@@
 	4025 4750 7650 4750
 $Comp
-L C-RESCUE-xmobile C?
+L xmobile-rescue:C-RESCUE-xmobile C?
 U 1 1 5C6D694B
 P 5650 2450
@@
 $EndComp
 $Comp
-L C-RESCUE-xmobile C?
+L xmobile-rescue:C-RESCUE-xmobile C?
 U 1 1 5C6D6A3D
 P 5650 2950
@@
 $EndComp
 $Comp
-L C-RESCUE-xmobile C?
+L xmobile-rescue:C-RESCUE-xmobile C?
 U 1 1 5C6D6B0E
 P 6150 2450
@@
 $EndComp
 $Comp
-L C-RESCUE-xmobile C?
+L xmobile-rescue:C-RESCUE-xmobile C?
 U 1 1 5C6D6B9B
 P 6150 2950
@@
 $EndComp
 $Comp
-L C-RESCUE-xmobile C?
+L xmobile-rescue:C-RESCUE-xmobile C?
 U 1 1 5C6D6CC6
 P 5900 4500
@@
 $EndComp
 $Comp
-L C-RESCUE-xmobile C?
+L xmobile-rescue:C-RESCUE-xmobile C?
 U 1 1 5C6D6D99
 P 6400 4500
@@
 $EndComp
 $Comp
-L C-RESCUE-xmobile C?
+L xmobile-rescue:C-RESCUE-xmobile C?
 U 1 1 5C6D6EE0
 P 5900 5000
@@
 $EndComp
 $Comp
-L C-RESCUE-xmobile C?
+L xmobile-rescue:C-RESCUE-xmobile C?
 U 1 1 5C6D6F6B
 P 5900 5500
@@
 $EndComp
 $Comp
-L C-RESCUE-xmobile C?
+L xmobile-rescue:C-RESCUE-xmobile C?
 U 1 1 5C6D7042
 P 6400 5000
@@
 $EndComp
 $Comp
-L C-RESCUE-xmobile C?
+L xmobile-rescue:C-RESCUE-xmobile C?
 U 1 1 5C6D70D1
 P 6400 5500
@@
 $EndComp
 $Comp
-L C-RESCUE-xmobile C?
+L xmobile-rescue:C-RESCUE-xmobile C?
 U 1 1 5C6D7206
 P 4025 4500
@@
 $EndComp
 $Comp
-L C-RESCUE-xmobile C?
+L xmobile-rescue:C-RESCUE-xmobile C?
 U 1 1 5C6D72FB
 P 4025 5000
@@
 $EndComp
 $Comp
-L C-RESCUE-xmobile C?
+L xmobile-rescue:C-RESCUE-xmobile C?
 U 1 1 5C6D7388
 P 4025 5500
@@
 $EndComp
 $Comp
-L C-RESCUE-xmobile C?
+L xmobile-rescue:C-RESCUE-xmobile C?
 U 1 1 5C6D77F5
 P 4525 4500
@@
 $EndComp
 $Comp
-L C-RESCUE-xmobile C?
+L xmobile-rescue:C-RESCUE-xmobile C?
 U 1 1 5C6D78F0
 P 4525 5000
@@
 $EndComp
 $Comp
-L C-RESCUE-xmobile C?
+L xmobile-rescue:C-RESCUE-xmobile C?
 U 1 1 5C6D7979
 P 4525 5500
@@
 $EndComp
 $Comp
-L LED-RESCUE-xmobile D?
+L xmobile-rescue:LED-RESCUE-xmobile D?
 U 1 1 5C6C7622
 P 7100 1900
@@
 $EndComp
 $Comp
-L LED-RESCUE-xmobile D?
+L xmobile-rescue:LED-RESCUE-xmobile D?
 U 1 1 5C6C77F4
 P 7100 3000
@@
 $EndComp
 $Comp
-L LED-RESCUE-xmobile D?
+L xmobile-rescue:LED-RESCUE-xmobile D?
 U 1 1 5C6C796F
 P 6725 3000
@@
 $EndComp
 $Comp
-L LED-RESCUE-xmobile D?
+L xmobile-rescue:LED-RESCUE-xmobile D?
 U 1 1 5C6C7BA9
 P 6975 4450
@@
 $EndComp
 $Comp
-L LED-RESCUE-xmobile D?
+L xmobile-rescue:LED-RESCUE-xmobile D?
 U 1 1 5C6C7D73
 P 7350 4450
@@
 $EndComp
 $Comp
-L LED-RESCUE-xmobile D?
+L xmobile-rescue:LED-RESCUE-xmobile D?
 U 1 1 5C6C7FDB
 P 7350 5550
@@
 $EndComp
 $Comp
-L LED-RESCUE-xmobile D?
+L xmobile-rescue:LED-RESCUE-xmobile D?
 U 1 1 5C6C809E
 P 6975 5550
