File: druid/xmobile_sim_holder.sch (KiCad schematic (older format))
At the start: 8 parts, among them U3 MOLEX_SIM_HOLDER_47553

Commit message: - Переделана клавиатура - установлены все корпуса микросхем
Parts:
- C22, C23: footprint (none) -> Capacitors_SMD:C_1206_HandSoldering; symbol C -> C-RESCUE-xmobile
- D10: footprint (none) -> semtech:SOT363
- R17, R18, R19, R20: footprint (none) -> Resistors_SMD:R_0603_HandSoldering; symbol R -> R-RESCUE-xmobile
- U3: footprint (none) -> molex:MOLEX_SIM_HOLDER_47553
Changed lines of the file:
@@
 EESchema Schematic File Version 2
+LIBS:xmobile-rescue
 LIBS:power
 LIBS:device
@@
 LIBS:contrib
 LIBS:valves
-LIBS:zakadc
-LIBS:vw2500m
-LIBS:usb-b
-LIBS:uprojects-msp430
-LIBS:uprojects-maxim-integrated
-LIBS:tps79530
-LIBS:tps63001
-LIBS:tps61040dbv
-LIBS:tact_sw
-LIBS:str751fr0t6
-LIBS:stm32f103cb
-LIBS:stm32f101cbt6
-LIBS:stm32f030f4
-LIBS:stm32f20x_LQFP64
-LIBS:sn54ac04
-LIBS:smf05c
-LIBS:sim_holder
-LIBS:sim900
-LIBS:sim800c
-LIBS:reset_supervisor
-LIBS:quectel
-LIBS:psl-ecg_12md_ads1298
-LIBS:pl2303
-LIBS:pcf8563_rtc
-LIBS:opa333_sot23-5
-LIBS:nrf8001
-LIBS:ncp3020
-LIBS:mt3608
-LIBS:molex_sim_holder_47553
-LIBS:micro_usb_b
-LIBS:microsd_socket
-LIBS:md1506_gsm_ant
-LIBS:mcp73833
-LIBS:mcp73831
-LIBS:mb6s
-LIBS:max669
-LIBS:ltc4120
-LIBS:ltc3533
-LIBS:lt1370
-LIBS:lpc1313
-LIBS:lp2951
-LIBS:lm2931cdr2g
-LIBS:lm809
-LIBS:lis3dh
-LIBS:led_couple
-LIBS:l6984
-LIBS:itg3200
-LIBS:irfh9310
-LIBS:irfh5300
-LIBS:ir2110l4
-LIBS:hmc5883
-LIBS:hlk-rm04
-LIBS:hc735-oscillator
-LIBS:gl850g_usb_hub
-LIBS:esp-07
-LIBS:dpak-diode
-LIBS:cstce_crystal
-LIBS:conn15
-LIBS:cc3100mod
-LIBS:bmp180
-LIBS:ble112
-LIBS:alt_symbols
-LIBS:ads1298_ecg_adc
-LIBS:ad8542
-LIBS:ad8495
-LIBS:ad8054
-LIBS:ad8051
-LIBS:3225_4p_quartz
-LIBS:74lvc02
 LIBS:XC6206P332MR
 LIBS:STF202-22T1G
 LIBS:MCP73871
+LIBS:switch1
 LIBS:xmobile-cache
 EELAYER 25 0
@@
 F 0 "U3" H 6200 3400 60  0000 C CNN
 F 1 "MOLEX_SIM_HOLDER_47553" H 6175 3275 60  0000 C CNN
-F 2 "" H 6125 2925 60  0000 C CNN
+F 2 "molex:MOLEX_SIM_HOLDER_47553" H 6125 2925 60  0000 C CNN
 F 3 "" H 6125 2925 60  0000 C CNN
 	1    6150 2950
@@
 F 0 "D10" H 5225 4225 60  0000 C CNN
 F 1 "SMF05C" H 4950 4225 60  0000 C CNN
-F 2 "" H 5115 4000 60  0000 C CNN
+F 2 "semtech:SOT363" H 5115 4000 60  0000 C CNN
 F 3 "" H 5115 4000 60  0000 C CNN
 	1    5125 4000
@@
 $EndComp
 $Comp
-L R R18
+L R-RESCUE-xmobile R18
 U 1 1 5A9F7A8D
 P 4425 3425
 F 0 "R18" V 4505 3425 40  0000 C CNN
 F 1 "51Omh" V 4432 3426 40  0000 C CNN
-F 2 "" V 4355 3425 30  0000 C CNN
+F 2 "Resistors_SMD:R_0603_HandSoldering" V 4355 3425 30  0000 C CNN
 F 3 "" H 4425 3425 30  0000 C CNN
 	1    4425 3425
@@
 $EndComp
 $Comp
-L C C22
+L C-RESCUE-xmobile C22
 U 1 1 5A9F7A94
 P 4000 3750
 F 0 "C22" H 4000 3850 40  0000 L CNN
 F 1 "22pF" H 4006 3665 40  0000 L CNN
-F 2 "" H 4038 3600 30  0000 C CNN
+F 2 "Capacitors_SMD:C_1206_HandSoldering" H 4038 3600 30  0000 C CNN
 F 3 "" H 4000 3750 60  0000 C CNN
 	1    4000 3750
@@
 NoConn ~ 6725 2900
 $Comp
-L R R19
+L R-RESCUE-xmobile R19
 U 1 1 5A9F7AA1
 P 4675 3000
 F 0 "R19" V 4755 3000 40  0000 C CNN
 F 1 "51Omh" V 4682 3001 40  0000 C CNN
-F 2 "" V 4605 3000 30  0000 C CNN
+F 2 "Resistors_SMD:R_0603_HandSoldering" V 4605 3000 30  0000 C CNN
 F 3 "" H 4675 3000 30  0000 C CNN
 	1    4675 3000
@@
 $EndComp
 $Comp
-L R R20
+L R-RESCUE-xmobile R20
 U 1 1 5A9F7AA8
 P 4875 2900
 F 0 "R20" V 4825 2700 40  0000 C CNN
 F 1 "51Omh" V 4882 2901 40  0000 C CNN
-F 2 "" V 4805 2900 30  0000 C CNN
+F 2 "Resistors_SMD:R_0603_HandSoldering" V 4805 2900 30  0000 C CNN
 F 3 "" H 4875 2900 30  0000 C CNN
 	1    4875 2900
@@
 $EndComp
 $Comp
-L R R17
+L R-RESCUE-xmobile R17
 U 1 1 5A9F7AB2
 P 3450 2925
 F 0 "R17" V 3530 2925 40  0000 C CNN
 F 1 "4.7KOmh" V 3457 2926 40  0000 C CNN
-F 2 "" V 3380 2925 30  0000 C CNN
+F 2 "Resistors_SMD:R_0603_HandSoldering" V 3380 2925 30  0000 C CNN
 F 3 "" H 3450 2925 30  0000 C CNN
 	1    3450 2925
@@
 $EndComp
 $Comp
-L C C23
+L C-RESCUE-xmobile C23
 U 1 1 5A9F7AB9
 P 5525 4200
 F 0 "C23" H 5525 4300 40  0000 L CNN
 F 1 "22pF" H 5531 4115 40  0000 L CNN
-F 2 "" H 5563 4050 30  0000 C CNN
+F 2 "Capacitors_SMD:C_1206_HandSoldering" H 5563 4050 30  0000 C CNN
 F 3 "" H 5525 4200 60  0000 C CNN
 	1    5525 4200

Commit message: Исправлины все ошибки и предупреждения в электрической схеме
Parts:
- added R27, R28: 0Omh, Resistors_SMD:R_0603_HandSoldering, symbol R-RESCUE-xmobile
Connections:
- net labels removed: GND_
- wire segments 19 -> 20
- no-connect marks 1 -> 2
Other:
- moved on the sheet: C22, C23, D10, R17, R18, R19, R20
Changed lines of the file:
@@
 L MOLEX_SIM_HOLDER_47553 U3
 U 1 1 5A9F7A7E
-P 6150 2950
-F 0 "U3" H 6200 3400 60  0000 C CNN
-F 1 "MOLEX_SIM_HOLDER_47553" H 6175 3275 60  0000 C CNN
-F 2 "molex:MOLEX_SIM_HOLDER_47553" H 6125 2925 60  0000 C CNN
-F 3 "" H 6125 2925 60  0000 C CNN
-	1    6150 2950
+P 6250 2950
+F 0 "U3" H 6300 3400 60  0000 C CNN
+F 1 "MOLEX_SIM_HOLDER_47553" H 6275 3275 60  0000 C CNN
+F 2 "molex:MOLEX_SIM_HOLDER_47553" H 6225 2925 60  0000 C CNN
+F 3 "" H 6225 2925 60  0000 C CNN
+	1    6250 2950
 	1    0    0    -1
 $EndComp
@@
 L SMF05C D10
 U 1 1 5A9F7A85
-P 5125 4000
-F 0 "D10" H 5225 4225 60  0000 C CNN
-F 1 "SMF05C" H 4950 4225 60  0000 C CNN
-F 2 "semtech:SOT363" H 5115 4000 60  0000 C CNN
-F 3 "" H 5115 4000 60  0000 C CNN
-	1    5125 4000
+P 5225 4000
+F 0 "D10" H 5325 4225 60  0000 C CNN
+F 1 "SMF05C" H 5050 4225 60  0000 C CNN
+F 2 "semtech:SOT363" H 5215 4000 60  0000 C CNN
+F 3 "" H 5215 4000 60  0000 C CNN
+	1    5225 4000
 	0    1    1    0
 $EndComp
@@
 L R-RESCUE-xmobile R18
 U 1 1 5A9F7A8D
-P 4425 3425
-F 0 "R18" V 4505 3425 40  0000 C CNN
-F 1 "51Omh" V 4432 3426 40  0000 C CNN
-F 2 "Resistors_SMD:R_0603_HandSoldering" V 4355 3425 30  0000 C CNN
-F 3 "" H 4425 3425 30  0000 C CNN
-	1    4425 3425
+P 4525 3425
+F 0 "R18" V 4605 3425 40  0000 C CNN
+F 1 "51Omh" V 4532 3426 40  0000 C CNN
+F 2 "Resistors_SMD:R_0603_HandSoldering" V 4455 3425 30  0000 C CNN
+F 3 "" H 4525 3425 30  0000 C CNN
+	1    4525 3425
 	0    1    1    0
 $EndComp
@@
 L C-RESCUE-xmobile C22
 U 1 1 5A9F7A94
-P 4000 3750
-F 0 "C22" H 4000 3850 40  0000 L CNN
-F 1 "22pF" H 4006 3665 40  0000 L CNN
-F 2 "Capacitors_SMD:C_1206_HandSoldering" H 4038 3600 30  0000 C CNN
-F 3 "" H 4000 3750 60  0000 C CNN
-	1    4000 3750
+P 4100 3750
+F 0 "C22" H 4100 3850 40  0000 L CNN
+F 1 "22pF" H 4106 3665 40  0000 L CNN
+F 2 "Capacitors_SMD:C_1206_HandSoldering" H 4138 3600 30  0000 C CNN
+F 3 "" H 4100 3750 60  0000 C CNN
+	1    4100 3750
 	1    0    0    -1
 $EndComp
-NoConn ~ 6725 2900
+NoConn ~ 6825 2900
 $Comp
 L R-RESCUE-xmobile R19
 U 1 1 5A9F7AA1
-P 4675 3000
-F 0 "R19" V 4755 3000 40  0000 C CNN
-F 1 "51Omh" V 4682 3001 40  0000 C CNN
-F 2 "Resistors_SMD:R_0603_HandSoldering" V 4605 3000 30  0000 C CNN
-F 3 "" H 4675 3000 30  0000 C CNN
-	1    4675 3000
+P 4775 3000
+F 0 "R19" V 4855 3000 40  0000 C CNN
+F 1 "51Omh" V 4782 3001 40  0000 C CNN
+F 2 "Resistors_SMD:R_0603_HandSoldering" V 4705 3000 30  0000 C CNN
+F 3 "" H 4775 3000 30  0000 C CNN
+	1    4775 3000
 	0    1    1    0
 $EndComp
@@
 L R-RESCUE-xmobile R20
 U 1 1 5A9F7AA8
-P 4875 2900
-F 0 "R20" V 4825 2700 40  0000 C CNN
-F 1 "51Omh" V 4882 2901 40  0000 C CNN
-F 2 "Resistors_SMD:R_0603_HandSoldering" V 4805 2900 30  0000 C CNN
-F 3 "" H 4875 2900 30  0000 C CNN
-	1    4875 2900
+P 4975 2900
+F 0 "R20" V 4925 2700 40  0000 C CNN
+F 1 "51Omh" V 4982 2901 40  0000 C CNN
+F 2 "Resistors_SMD:R_0603_HandSoldering" V 4905 2900 30  0000 C CNN
+F 3 "" H 4975 2900 30  0000 C CNN
+	1    4975 2900
 	0    1    1    0
 $EndComp
@@
 L R-RESCUE-xmobile R17
 U 1 1 5A9F7AB2
-P 3450 2925
-F 0 "R17" V 3530 2925 40  0000 C CNN
-F 1 "4.7KOmh" V 3457 2926 40  0000 C CNN
-F 2 "Resistors_SMD:R_0603_HandSoldering" V 3380 2925 30  0000 C CNN
-F 3 "" H 3450 2925 30  0000 C CNN
-	1    3450 2925
+P 2400 2925
+F 0 "R17" V 2480 2925 40  0000 C CNN
+F 1 "4.7KOmh" V 2407 2926 40  0000 C CNN
+F 2 "Resistors_SMD:R_0603_HandSoldering" V 2330 2925 30  0000 C CNN
+F 3 "" H 2400 2925 30  0000 C CNN
+	1    2400 2925
 	0    1    1    0
 $EndComp
@@
 L C-RESCUE-xmobile C23
 U 1 1 5A9F7AB9
-P 5525 4200
-F 0 "C23" H 5525 4300 40  0000 L CNN
-F 1 "22pF" H 5531 4115 40  0000 L CNN
-F 2 "Capacitors_SMD:C_1206_HandSoldering" H 5563 4050 30  0000 C CNN
-F 3 "" H 5525 4200 60  0000 C CNN
-	1    5525 4200
+P 5625 4200
+F 0 "C23" H 5625 4300 40  0000 L CNN
+F 1 "22pF" H 5631 4115 40  0000 L CNN
+F 2 "Capacitors_SMD:C_1206_HandSoldering" H 5663 4050 30  0000 C CNN
+F 3 "" H 5625 4200 60  0000 C CNN
+	1    5625 4200
 	1    0    0    -1
 $EndComp
 Wire Wire Line
-	7000 3425 4675 3425
+	7100 3425 4775 3425
 Wire Wire Line
-	4825 3425 4825 3775
+	4925 3425 4925 3775
 Wire Wire Line
-	3900 3425 4175 3425
+	4000 3425 4275 3425
 Wire Wire Line
-	4000 3425 4000 3550
-Connection ~ 4000 3425
-Connection ~ 4825 3425
+	4100 3425 4100 3550
+Connection ~ 4100 3425
+Connection ~ 4925 3425
 Wire Wire Line
-	6725 3000 7000 3000
+	6825 3000 7100 3000
 Wire Wire Line
-	7000 2800 7000 3425
+	3950 3100 5725 3100
 Wire Wire Line
-	3250 3200 5625 3200
+	5025 3775 5025 3200
+Connection ~ 5025 3200
 Wire Wire Line
-	5625 3100 5425 3100
+	5325 3775 5325 2800
+Connection ~ 5325 2800
 Wire Wire Line
-	5425 3100 5425 3200
-Connection ~ 5425 3200
+	5125 3775 5125 3000
+Connection ~ 5125 3000
 Wire Wire Line
-	6725 2800 7000 2800
-Connection ~ 7000 3000
+	5150 2800 5725 2800
 Wire Wire Line
-	4925 3775 4925 3200
-Connection ~ 4925 3200
+	5225 2900 5725 2900
 Wire Wire Line
-	5225 3775 5225 2800
-Connection ~ 5225 2800
+	5025 3000 5725 3000
 Wire Wire Line
-	5025 3775 5025 3000
-Connection ~ 5025 3000
+	2650 2925 2700 2925
 Wire Wire Line
-	5050 2800 5625 2800
+	2700 2925 2700 3200
+Connection ~ 2700 3200
 Wire Wire Line
-	5125 2900 5625 2900
+	5625 4000 5625 2800
+Connection ~ 5625 2800
+Text HLabel 5150 2800 0    60   Input ~ 0
+SIM_VCC
+Text HLabel 4725 2900 0    60   Input ~ 0
+SIM_RST
+Text HLabel 4525 3000 0    60   Input ~ 0
+SIM_CLK
+Text HLabel 5200 2100 0    60   BiDi ~ 0
+GND
+Text HLabel 2150 2925 0    60   Input ~ 0
+GSM_VDD
+Text HLabel 2200 3200 0    60   Output ~ 0
+SIM_DET
+Text HLabel 4000 3425 0    60   BiDi ~ 0
+SIM_DATA
+Text Label 5200 2100 0    60   ~ 0
+GND
+Text Label 6825 3100 0    60   ~ 0
+GND
+Text Label 5625 4400 3    60   ~ 0
+GND
+Text Label 5125 4375 3    60   ~ 0
+GND
+Text Label 4100 3950 3    60   ~ 0
+GND
+$Comp
+L R-RESCUE-xmobile R27
+U 1 1 5AB7668E
+P 3175 3200
+F 0 "R27" V 3255 3200 40  0000 C CNN
+F 1 "0Omh" V 3182 3201 40  0000 C CNN
+F 2 "Resistors_SMD:R_0603_HandSoldering" V 3105 3200 30  0000 C CNN
+F 3 "" H 3175 3200 30  0000 C CNN
+	1    3175 3200
+	0    1    1    0
+$EndComp
+$Comp
+L R-RESCUE-xmobile R28
+U 1 1 5AB7B1D6
+P 3700 3100
+F 0 "R28" V 3780 3100 40  0000 C CNN
+F 1 "0Omh" V 3707 3101 40  0000 C CNN
+F 2 "Resistors_SMD:R_0603_HandSoldering" V 3630 3100 30  0000 C CNN
+F 3 "" H 3700 3100 30  0000 C CNN
+	1    3700 3100
+	0    1    1    0
+$EndComp
 Wire Wire Line
-	4925 3000 5625 3000
+	3450 3100 2825 3100
 Wire Wire Line
-	3700 2925 3750 2925
+	2825 3100 2825 3200
+Connection ~ 2825 3200
 Wire Wire Line
-	3750 2925 3750 3200
-Connection ~ 3750 3200
+	5725 3200 3425 3200
 Wire Wire Line
-	5525 4000 5525 2800
-Connection ~ 5525 2800
-Text HLabel 5050 2800 0    60   Input ~ 0
-SIM_VCC
-Text HLabel 4625 2900 0    60   Input ~ 0
-SIM_RST
-Text HLabel 4425 3000 0    60   Input ~ 0
-SIM_CLK
-Text HLabel 5100 2100 0    60   BiDi ~ 0
+	2200 3200 2925 3200
+NoConn ~ 5225 3775
+Text Label 6825 2800 0    60   ~ 0
 GND
-Text HLabel 3200 2925 0    60   Input ~ 0
-GSM_VDD
-Text HLabel 3250 3200 0    60   Output ~ 0
-SIM_DET
-Text HLabel 3900 3425 0    60   BiDi ~ 0
-SIM_DATA
-Text Label 5100 2100 0    60   ~ 0
-GND_
-Text Label 6725 3100 0    60   ~ 0
-GND_
-Text Label 5525 4400 3    60   ~ 0
-GND_
-Text Label 5025 4375 3    60   ~ 0
-GND_
-Text Label 4000 3950 3    60   ~ 0
-GND_
+Wire Wire Line
+	7100 3000 7100 3425
 $EndSCHEMATC

Commit message: Add 6 pin SIM holder (add pdf) Connect SIM800C to sim holder
Parts:
- added C? (x2): 22pF, Capacitors_SMD:C_1206_HandSoldering, symbol C-RESCUE-xmobile
- added D?: SMF05C, semtech:SOT363, symbol SMF05C
- added R? (x4): 51Omh, Resistors_SMD:R_0603_HandSoldering, symbol R-RESCUE-xmobile
- added U?: SIM800C, symbol SIM800C
- added U?: 78646-3001, symbol 78646-3001
Connections:
- net labels added: SIM_VDD
- wire segments 20 -> 40
Changed lines of the file:
@@
 LIBS:SRAM
 LIBS:xmega128a1u_bga100
+LIBS:sim-holders
 LIBS:xmobile-cache
 EELAYER 25 0
@@
 Wire Wire Line
 	7100 3000 7100 3425
+$Comp
+L SIM800C U?
+U 1 1 5C46A8F4
+P 9400 3825
+F 0 "U?" H 9450 4800 60  0000 C CNN
+F 1 "SIM800C" H 8750 4800 60  0000 C CNN
+F 2 "" H 9400 3825 60  0000 C CNN
+F 3 "" H 9400 3825 60  0000 C CNN
+	1    9400 3825
+	1    0    0    -1
+$EndComp
+$Comp
+L 78646-3001 U?
+U 1 1 5C46ADE6
+P 5175 5550
+F 0 "U?" H 5275 5350 60  0000 C CNN
+F 1 "78646-3001" H 5325 5500 60  0000 C CNN
+F 2 "" H 5175 5600 60  0000 C CNN
+F 3 "" H 5175 5600 60  0000 C CNN
+	1    5175 5550
+	1    0    0    -1
+$EndComp
+Text Label 1500 4850 2    60   ~ 0
+SIM_VDD
+Text Label 8350 4300 2    60   ~ 0
+SIM_VDD
+Text Label 8350 4150 2    60   ~ 0
+SIM_CLK
+Text Label 1525 5450 2    60   ~ 0
+SIM_CLK
+Text Label 8350 4225 2    60   ~ 0
+SIM_RST
+Text Label 1525 5150 2    60   ~ 0
+SIM_RST
+Text Label 8350 4525 2    60   ~ 0
+GND
+Text Label 4575 5600 2    60   ~ 0
+GND
+Text Label 8350 4075 2    60   ~ 0
+SIM_DATA
+Text Label 1500 5800 2    60   ~ 0
+SIM_DATA
+$Comp
+L SMF05C D?
+U 1 1 5C46C4AB
+P 3650 6425
+F 0 "D?" H 3750 6650 60  0000 C CNN
+F 1 "SMF05C" H 3475 6650 60  0000 C CNN
+F 2 "semtech:SOT363" H 3640 6425 60  0000 C CNN
+F 3 "" H 3640 6425 60  0000 C CNN
+	1    3650 6425
+	0    1    1    0
+$EndComp
+$Comp
+L R-RESCUE-xmobile R?
+U 1 1 5C46C6D5
+P 1925 5800
+F 0 "R?" V 2005 5800 40  0000 C CNN
+F 1 "51Omh" V 1932 5801 40  0000 C CNN
+F 2 "Resistors_SMD:R_0603_HandSoldering" V 1855 5800 30  0000 C CNN
+F 3 "" H 1925 5800 30  0000 C CNN
+	1    1925 5800
+	0    1    1    0
+$EndComp
+Wire Wire Line
+	2175 5800 4575 5800
+Wire Wire Line
+	3350 6200 3350 5800
+Connection ~ 3350 5800
+$Comp
+L C-RESCUE-xmobile C?
+U 1 1 5C46CACB
+P 2325 6400
+F 0 "C?" H 2325 6500 40  0000 L CNN
+F 1 "22pF" H 2331 6315 40  0000 L CNN
+F 2 "Capacitors_SMD:C_1206_HandSoldering" H 2363 6250 30  0000 C CNN
+F 3 "" H 2325 6400 60  0000 C CNN
+	1    2325 6400
+	1    0    0    -1
+$EndComp
+Wire Wire Line
+	2325 6200 2325 5800
+Connection ~ 2325 5800
+$Comp
+L R-RESCUE-xmobile R?
+U 1 1 5C46D160
+P 1925 5450
+F 0 "R?" V 2005 5450 40  0000 C CNN
+F 1 "51Omh" V 1932 5451 40  0000 C CNN
+F 2 "Resistors_SMD:R_0603_HandSoldering" V 1855 5450 30  0000 C CNN
+F 3 "" H 1925 5450 30  0000 C CNN
+	1    1925 5450
+	0    1    1    0
+$EndComp
+$Comp
+L R-RESCUE-xmobile R?
+U 1 1 5C46D2D8
+P 1925 5150
+F 0 "R?" V 2005 5150 40  0000 C CNN
+F 1 "51Omh" V 1932 5151 40  0000 C CNN
+F 2 "Resistors_SMD:R_0603_HandSoldering" V 1855 5150 30  0000 C CNN
+F 3 "" H 1925 5150 30  0000 C CNN
+	1    1925 5150
+	0    1    1    0
+$EndComp
+$Comp
+L R-RESCUE-xmobile R?
+U 1 1 5C46D4E7
+P 1925 4850
+F 0 "R?" V 2005 4850 40  0000 C CNN
+F 1 "51Omh" V 1932 4851 40  0000 C CNN
+F 2 "Resistors_SMD:R_0603_HandSoldering" V 1855 4850 30  0000 C CNN
+F 3 "" H 1925 4850 30  0000 C CNN
+	1    1925 4850
+	0    1    1    0
+$EndComp
+Wire Wire Line
+	1525 5450 1675 5450
+Wire Wire Line
+	1675 5150 1525 5150
+Wire Wire Line
+	1675 4850 1500 4850
+Wire Wire Line
+	1500 5800 1675 5800
+Wire Wire Line
+	2175 5450 2400 5450
+Wire Wire Line
+	2400 5450 2400 5500
+Wire Wire Line
+	2400 5500 4575 5500
+Wire Wire Line
+	2175 5150 4400 5150
+Wire Wire Line
+	4400 5150 4400 5400
+Wire Wire Line
+	4400 5400 4575 5400
+Wire Wire Line
+	2175 4850 4500 4850
+Wire Wire Line
+	4500 4850 4500 5300
+Wire Wire Line
+	4500 5300 4575 5300
+Wire Wire Line
+	3550 6200 3550 5500
+Connection ~ 3550 5500
+Wire Wire Line
+	3650 6200 3650 5150
+Connection ~ 3650 5150
+Wire Wire Line
+	3750 6200 3750 4850
+Connection ~ 3750 4850
+Text Label 3550 6800 3    60   ~ 0
+GND
+$Comp
+L C-RESCUE-xmobile C?
+U 1 1 5C46E5BE
+P 3100 7125
+F 0 "C?" H 3100 7225 40  0000 L CNN
+F 1 "22pF" H 3106 7040 40  0000 L CNN
+F 2 "Capacitors_SMD:C_1206_HandSoldering" H 3138 6975 30  0000 C CNN
+F 3 "" H 3100 7125 60  0000 C CNN
+	1    3100 7125
+	1    0    0    -1
+$EndComp
+Wire Wire Line
+	3100 4850 3100 6925
+Connection ~ 3100 4850
+Text Label 3100 7325 3    60   ~ 0
+GND
 $EndSCHEMATC

Commit message: Design and connect GSM module.
Parts:
- removed C22, C23: 22pF, Capacitors_SMD:C_1206_HandSoldering, symbol C-RESCUE-xmobile
- removed D10: SMF05C, semtech:SOT363, symbol SMF05C
- removed R17: 4.7KOmh, Resistors_SMD:R_0603_HandSoldering, symbol R-RESCUE-xmobile
- removed R18, R19, R20: 51Omh, Resistors_SMD:R_0603_HandSoldering, symbol R-RESCUE-xmobile
- removed R27, R28: 0Omh, Resistors_SMD:R_0603_HandSoldering, symbol R-RESCUE-xmobile
- removed U3: MOLEX_SIM_HOLDER_47553, molex:MOLEX_SIM_HOLDER_47553, symbol MOLEX_SIM_HOLDER_47553
- added C?: 22pF, Capacitors_SMD:C_1206_HandSoldering, symbol C-RESCUE-xmobile
- added D?: LED, symbol LED
- added P?: USB_A, symbol USB_A
- added Q? (x2): BC850, SOT-23, symbol BC850
- added R? (x8): 1k, Resistors_SMD:R_0603_HandSoldering, symbol R-RESCUE-xmobile
- added R?: 47k, Resistors_SMD:R_0603_HandSoldering, symbol R-RESCUE-xmobile
- added R? (x2): 4.7K, Resistors_SMD:R_0603_HandSoldering, symbol R-RESCUE-xmobile
- added R?: 47K, Resistors_SMD:R_0603_HandSoldering, symbol R-RESCUE-xmobile
- added R? (x3): 5.6k, Resistors_SMD:R_0603_HandSoldering, symbol R-RESCUE-xmobile
- added U?: STF202-22T1G, MODULE, symbol STF202-22T1G
- added W?: TP_RTC_BAT, symbol TEST
- added W?: TP_GSM_ANT, symbol TEST_1P
- added W?: TP_BT_ANT, symbol TEST_1P
- added W?: TP_UART_RXD, symbol TEST_1P
- added W?: TP_UART_RTS, symbol TEST_1P
- added W?: TP_UART_DTR, symbol TEST_1P
- added W?: TP_UART_CTS, symbol TEST_1P
- added W?: TP_UART_DCD, symbol TEST_1P
- added W?: TP_UART_RI, symbol TEST_1P
- added W?: TP_USART_TXD, symbol TEST_1P
- R? (x4): value 51Omh -> 51
Connections:
- net labels added: GSM_VBAT, MICN, MICP, NETLIGHT, POWER_KEY, PWRKEY, SPKN, SPKP, STATUS, UART_CTS, UART_DCD, UART_DTR, UART_RI, UART_RTS, UART_RXD, UART_TXD, USB_DN, USB_DP, USB_VBUS
- net labels removed: GSM_VDD, SIM_DET, SIM_VCC
- wire segments 40 -> 73
- no-connect marks 2 -> 8
Other:
- note added: "Antenna TP should be close to module\nand far from power and sim holder."
- note added: "SIM800 power on:\npull PWRKEY down for a second and then pull it up.\nIt already pulled up to VBAT in the module internal."
- moved on the sheet: C?, D?, R?, U?

Commit message: Added microSD slot.
Parts:
- D?: symbol LED -> LED-RESCUE-xmobile
- P?: symbol USB_A -> USB_A-RESCUE-xmobile
- W?: symbol TEST -> TEST-RESCUE-xmobile
Connections:
- net GSM_VBAT: now also D?.2 (A)
- net at D?.1 (K): now also R?.2
- no-connect marks 8 -> 7
Changed lines of the file:
@@
 GSM_VBAT
 $Comp
-L LED D?
+L LED-RESCUE-xmobile D?
 U 1 1 5C46F9F6
 P 10425 3975
@@
 GND
 $Comp
-L TEST W?
+L TEST-RESCUE-xmobile W?
 U 1 1 5C481A0A
 P 7850 3775
@@
 NoConn ~ 7275 4150
 NoConn ~ 7275 4225
-NoConn ~ 8275 4200
 Text Label 7275 3025 0    60   ~ 0
 GSM_VBAT
@@
 $EndComp
 $Comp
-L USB_A P?
+L USB_A-RESCUE-xmobile P?
 U 1 1 5C499B15
 P 9925 1950
