File: druid/xmobile_sim_holder.sch (KiCad schematic (older format))
At the start: 40 parts

Commit message: looks like all packages added.
Parts:
- removed C? (x2): 22p, symbol xmobile-rescue:C-RESCUE-xmobile
- removed D?: LED, symbol xmobile-rescue:LED-RESCUE-xmobile
- removed Q?: BC850, SOT-23, symbol xmobile-rescue:BC850
- removed R? (x3): 51, symbol xmobile-rescue:R-RESCUE-xmobile
- removed R? (x8): 1k, symbol xmobile-rescue:R-RESCUE-xmobile
- removed R?: 4.7K, symbol xmobile-rescue:R-RESCUE-xmobile
- removed R?: 47K, symbol xmobile-rescue:R-RESCUE-xmobile
- added C? (x2): 22p, Capacitors_SMD:C_0402, symbol xmobile-rescue:C-RESCUE-xmobile
- added D?: LED WHITE, LEDs_git:LED_0402, symbol xmobile-rescue:LED-RESCUE-xmobile
- added Q?: BC850, SOT:SOT-23, symbol xmobile-rescue:BC850
- added R? (x8): 1k, Resistors_SMD:R_0402, symbol xmobile-rescue:R-RESCUE-xmobile
- added R?: 47k, Resistors_SMD:R_0402, symbol xmobile-rescue:R-RESCUE-xmobile
- added R?: 4.7K, Resistors_SMD:R_0402, symbol xmobile-rescue:R-RESCUE-xmobile
- added R? (x3): 51, Resistors_SMD:R_0402, symbol xmobile-rescue:R-RESCUE-xmobile
- C?: footprint (none) -> Capacitors_SMD:C_0402; case (none) -> 0402 In; example (none) -> https://www.mouser.co.uk/ProductDetail/Murata-Electronics/G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
- D?: case (none) -> SOT-363; example (none) -> https://www.mouser.co.uk/ProductDetail/ON-Semiconductor/SMF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
- P?: value USB_A -> microUSB; case (none) -> microUSB-B; example (none) -> https://www.mouser.co.uk/ProductDetail/Molex/47346-0001?qs=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
- Q?: footprint SOT-23 -> SOT:SOT-23; case (none) -> SOT-23; example (none) -> https://www.mouser.co.uk/ProductDetail/ON-Semiconductor-Fai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
- R?: footprint (none) -> Resistors_SMD:R_0402; case (none) -> 0402 In; example (none) -> https://www.mouser.co.uk/ProductDetail/Vishay/CRCW040251R0F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
- R?: footprint (none) -> Resistors_SMD:R_0402; case (none) -> 0402 In; example (none) -> https://www.mouser.co.uk/ProductDetail/Vishay/RCS040247K0FK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
- R?: footprint (none) -> Resistors_SMD:R_0402; case (none) -> 0402 In; example (none) -> https://www.mouser.co.uk/ProductDetail/Vishay/CRCW04024K70J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
- R?: footprint (none) -> Resistors_SMD:R_0402; case (none) -> 0402 In; example (none) -> https://www.mouser.co.uk/ProductDetail/Panasonic/ERJ-2RKF56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
- R?: footprint (none) -> Resistors_SMD:R_0402; case (none) -> 0402 In; example (none) -> https://www.mouser.co.uk/ProductDetail/Yageo/RC0402FR-075K6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
- U?: case (none) -> SIM800C LCC; example (none) -> https://ru.aliexpress.com/item/SIM800C-SIM800-Four-frequenc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
- U?: case (none) -> 6 pin microSIM; example (none) -> https://eu.mouser.com/ProductDetail/Molex/78646-3001?qs=%2f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
- U?: case (none) -> TSOP-6; example (none) -> https://www.mouser.co.uk/ProductDetail/ON-Semiconductor/STF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
- W?: footprint (none) -> Measurement_Points:Test_Point_2Pads; case (none) -> 2 pads
- W? (x9): footprint (none) -> Measurement_Points:Measurement_Point_Square-TH_Small; case (none) -> 1 pad
Connections:
- net GND: now also C?.2, C?.2, Q?.2 (E), R?.2
- net GSM_VBAT: now also D?.2 (A)
- net NETLIGHT: now also R?.1
- net SIM_CLK: now also R?.2
- net SIM_DATA: now also R?.2
- net SIM_RST: now also R?.2
- net UART_CTS: now also R?.2
- net UART_DCD: now also R?.2
- net UART_DTR: now also R?.2
- net UART_RI: now also R?.2
- net UART_RTS: now also R?.2
- net UART_RXD: now also R?.1
- net UART_TXD: now also R?.1
- net USB_VBUS: now also C?.1
- net at U?.1 (UART1_TXD): now also R?.2
- net at R?.2, U?.2 (UART1_RXD): now also R?.2
- net at R?.2, U?.3 (UART1_RTS): now also R?.1
- net at U?.4 (UART1_CTS): now also R?.1
- net at U?.5 (UART1_DCD): now also R?.1
- net at R?.2, U?.6 (UART1_DTR): now also R?.1
- net at U?.7 (UART1_RI): now also R?.1
- net at D?.1, R?.1, U?.1 (VCC): now also C?.1
- net at D?.3, U?.2 (RST): now also R?.1
- net at D?.4, U?.3 (CLK): now also R?.1
- net at C?.1, D?.6, U?.7 (IO): now also R?.1
- net at R?.2: now also Q?.1 (B), R?.2
- net at Q?.1 (B), R?.2: now also R?.1
- new net: Q?.3 (C), R?.1
- new net: D?.1 (K), R?.2
