File: druid/xmobile_sim_holder.sch (KiCad schematic (older format))
At the start: 40 parts

Commit message: remove electric  warnings and errors. annotate elements. fix microUSB-B symbol.
Parts:
- removed P?: microUSB, Connectors_USB:USB_Micro-B_Molex_47346-0001, symbol xmobile-rescue:USB_A-RESCUE-xmobile
- added J4: USB_B_Micro, Connectors_USB:USB_Micro-B_Molex_47346-0001, symbol Connector:USB_B_Micro
- gave numbers to parts that had none: 39
Connections:
- net USB_DN: now also U9.2 (D(IN)); no longer U9.3 (D(IN))
- net USB_DP: now also U9.3 (D(IN)); no longer U9.1 (VBUS)
- net USB_VBUS: now also U9.1 (VBUS), J4.1 (VBUS); no longer U9.2 (D(IN))
- net at U9.4 (D(OUT)): now also J4.3 (D+)
- net at U9.5 (D(OUT)): now also J4.2 (D-)
- net at U9.6 (GND): now also J4.4 (ID), J4.5 (GND), J4.6 (Shield)
- net GSM_VBAT renamed 3.7V
Other:
- moved on the sheet: C34, U9

Commit message: Some small fixes. generated net list.
Parts:
- R22: footprint (none) -> Resistors_SMD:R_0402; case (none) -> 0402 In; example (none) -> https://www.mouser.co.uk/ProductDetail/Panasonic/ERA-2AEB56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
Changed lines of the file:
@@
 F 0 "R22" V 3680 3100 40  0000 C CNN
 F 1 "5.6k" V 3607 3101 40  0000 C CNN
-F 2 "" V 3530 3100 30  0000 C CNN
-F 3 "" H 3600 3100 30  0000 C CNN
+F 2 "Resistors_SMD:R_0402" V 3530 3100 30  0001 C CNN
+F 3 "https://www.mouser.co.uk/datasheet/2/315/AOA0000C307-1149632.pdf" H 3600 3100 30  0001 C CNN
+F 4 "https://www.mouser.co.uk/ProductDetail/Panasonic/ERA-2AEB562X?qs=sGAEpiMZZMtlubZbdhIBILRDuhBknqQkIY4D4uMGNNo%3d" V 3600 3100 50  0001 C CNN "example"
+F 5 "0402 In" V 3525 3100 30  0000 C CNN "case"
 	1    3600 3100
 	-1   0    0    1

Commit message: fix U1 package pin names
Parts:
- D18: footprint semtech:SOT363 -> TO_SOT_Packages_SMD:SOT-363_SC-70-6
- J4: symbol Connector:USB_B_Micro -> xmobile-rescue:USB_B_Micro-Connector
Changed lines of the file:
@@
 U 1 1 5C46C4AB
 P 3250 6650
-F 0 "D18" V 3325 6875 60  0000 C CNN
+F 0 "D18" V 3325 6925 60  0000 C CNN
 F 1 "SMF05C" V 3500 6750 60  0000 C CNN
-F 2 "semtech:SOT363" H 3250 6975 60  0001 C CNN
+F 2 "TO_SOT_Packages_SMD:SOT-363_SC-70-6" H 3250 6975 60  0001 C CNN
 F 3 "https://www.mouser.co.uk/datasheet/2/308/SMF05C-D-100912.pdf" H 3240 6650 60  0001 C CNN
 F 4 "https://www.mouser.co.uk/ProductDetail/ON-Semiconductor/SMF05CT1G?qs=sGAEpiMZZMtqO%252bWUGLBzeAEUVu%2fYzK%252bE" H 3250 6650 50  0001 C CNN "example"
@@
 	1100 5075 1275 5075
 $Comp
-L Connector:USB_B_Micro J4
+L xmobile-rescue:USB_B_Micro-Connector J4
 U 1 1 5C70D478
 P 10200 1325
+AR Path="/5C70D478" Ref="J4"  Part="1"
+AR Path="/5A9F76AF/5C70D478" Ref="J4"  Part="1"
 F 0 "J4" H 9971 1193 50  0000 R CNN
 F 1 "USB_B_Micro" H 9971 1284 50  0000 R CNN

Commit message: fix other packages. Start doing layout
Parts:
- C32, C33, C34: footprint Capacitors_SMD:C_0402 -> Capacitor_SMD:C_0402_1005Metric
- D18: footprint TO_SOT_Packages_SMD:SOT-363_SC-70-6 -> Package_TO_SOT_SMD:SOT-363_SC-70-6
- D19: footprint LEDs_git:LED_0402 -> LED_SMD:LED_0402_1005Metric
- J4: footprint Connectors_USB:USB_Micro-B_Molex_47346-0001 -> Connector_USB:USB_Micro-B_Molex_47346-0001
- Q1, Q2: footprint SOT:SOT-23 -> Package_TO_SOT_SMD:SOT-23
- R15, R16, R17, R18, R19, R20, R21, R22, R23, R24, R25, R26, R27, R28, R29, R30, R31, R32, R33: footprint Resistors_SMD:R_0402 -> Resistor_SMD:R_0402_1005Metric
- W10, W11, W12, W13, W14, W15, W16, W18, W9: footprint Measurement_Points:Measurement_Point_Square-TH_Small -> TestPoint:TestPoint_THTPad_1.0x1.0mm_Drill0.5mm
- W17: footprint Measurement_Points:Test_Point_2Pads -> TestPoint:TestPoint_2Pads_Pitch2.54mm_Drill0.8mm
