File: druid/xmobile.sch (KiCad schematic (older format))
At the start: 44 parts, among them CON1 AVR-PDI-6, IC1 ATXMEGA128A1U-A, P1 USB_B, P10 CONN_01X08, P2 CONN_01X02, P3 CONN_8, P7 CONN_4, Q1 A2SHB, Q2 A2SHB, U1 STF202-22T1G, U2 SIM800C, U5 switch1

Commit message: [XMEGA] Add BGA xmega electrical lib, SRAM connected (no power capacitors)
Parts:
- added U?: XMega128A1U_BGA100, symbol XMega128A1U_BGA100
Connections:
- net labels added: +3.3V_filtered, A0, A1, A10, A11, A12, A13, A14, A15, A16, A17, A18, A19, A2, A3, A4, A5, A6, A7, A8, A9, CE1, CE2, D0, D1, D2, D3, D4, D5, D6, D7, OE, WE
- wire segments 75 -> 77
Other:
- moved on the sheet: C1, C2, C3, C32, C33, C34, C35, C36, C37, C38, C39, C40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

Commit message: Add 6 pin SIM holder (add pdf) Connect SIM800C to sim holder
Connections:
- wire segments 77 -> 106
Other:
- moved on the sheet: U2
Changed lines of the file:
@@
 LIBS:SRAM
 LIBS:xmega128a1u_bga100
+LIBS:sim-holders
 LIBS:xmobile-cache
 EELAYER 25 0
@@
 L SIM800C U2
 U 1 1 59667E03
-P 30250 17650
-F 0 "U2" H 30300 18625 60  0000 C CNN
-F 1 "SIM800C" H 29600 18625 60  0000 C CNN
-F 2 "SIM800C_lup:SIM800C" H 30075 17850 60  0000 C CNN
-F 3 "" H 30250 17650 60  0000 C CNN
-	1    30250 17650
+P 18725 16350
+F 0 "U2" H 18775 17325 60  0000 C CNN
+F 1 "SIM800C" H 18075 17325 60  0000 C CNN
+F 2 "SIM800C_lup:SIM800C" H 18550 16550 60  0000 C CNN
+F 3 "" H 18725 16350 60  0000 C CNN
+	1    18725 16350
 	1    0    0    -1
 $EndComp
@@
 	0    -1   -1   0
 $EndComp
-Text Label 29200 17375 2    60   ~ 0
-GND
-Text Label 29200 17750 2    60   ~ 0
-GND
-Text Label 29200 18200 2    60   ~ 0
-GND
-Text Label 29200 18350 2    60   ~ 0
-GND
-Text Label 30900 17525 0    60   ~ 0
-GND
-Text Label 30900 17750 0    60   ~ 0
-GND
-Text Label 30900 17225 0    60   ~ 0
-GND
-Text Label 30900 17450 0    60   ~ 0
+Text Label 17675 16075 2    60   ~ 0
+GND
+Text Label 17675 16450 2    60   ~ 0
+GND
+Text Label 17675 16900 2    60   ~ 0
+GND
+Text Label 17675 17050 2    60   ~ 0
+GND
+Text Label 19375 16225 0    60   ~ 0
+GND
+Text Label 19375 16450 0    60   ~ 0
+GND
+Text Label 19375 15925 0    60   ~ 0
+GND
+Text Label 19375 16150 0    60   ~ 0
 3.7V
-Text Label 30900 17375 0    60   ~ 0
+Text Label 19375 16075 0    60   ~ 0
 3.7V
-Text Label 30900 17975 0    60   ~ 0
-GND
-Text Label 30900 17675 0    60   ~ 0
+Text Label 19375 16675 0    60   ~ 0
+GND
+Text Label 19375 16375 0    60   ~ 0
 GND
 Text Label 10275 10100 0    60   ~ 0
@@
 Text Label 29800 13450 0    60   ~ 0
 XMEGA_PE0_GPIO
-Text Label 29200 17000 2    60   ~ 0
+Text Label 17675 15700 2    60   ~ 0
 GSM_AT_RTS
-Text Label 29200 16850 2    60   ~ 0
+Text Label 17675 15550 2    60   ~ 0
 GSM_AT_TXD
 Text Label 33800 16450 0    60   ~ 0
@@
 Text Label 29800 12900 0    60   ~ 0
 XMEGA_PD3_GPIO
-Text Label 29200 17150 2    60   ~ 0
+Text Label 17675 15850 2    60   ~ 0
 GSM_AT_DCD
-Text Label 29200 16925 2    60   ~ 0
+Text Label 17675 15625 2    60   ~ 0
 GSM_AT_RXD
 $Comp
@@
 Text Label 33800 16900 0    60   ~ 0
 XMEGA_PD1_GPIO
-Text Label 29200 17075 2    60   ~ 0
+Text Label 17675 15775 2    60   ~ 0
 GSM_AT_CTS
-Text Label 29200 17225 2    60   ~ 0
+Text Label 17675 15925 2    60   ~ 0
 GSM_AT_DTR
-Text Label 29200 17300 2    60   ~ 0
+Text Label 17675 16000 2    60   ~ 0
 GSM_AT_RI
 Text Label 29800 12700 0    60   ~ 0
@@
 	1    0    0    -1
 $EndComp
-Text Label 30900 18050 0    60   ~ 0
+Text Label 19375 16750 0    60   ~ 0
 GSM_USB_DN
 Text Label 21250 12425 2    60   ~ 0
 GSM_USB_DN
-Text Label 30900 18125 0    60   ~ 0
+Text Label 19375 16825 0    60   ~ 0
 GSM_USB_DP
 Text Label 21250 12525 2    60   ~ 0
@@
 Text Label 20600 11700 2    60   ~ 0
 GND
-Text Label 30900 18200 0    60   ~ 0
+Text Label 19375 16900 0    60   ~ 0
 GSM_USB_VBUS
 Text Label 21250 12325 2    60   ~ 0
 GSM_USB_VBUS
-Text Label 30900 16925 0    60   ~ 0
+Text Label 19375 15625 0    60   ~ 0
 GSM_NETLIGHT
 $Comp
@@
 Text Label 22475 15100 3    60   ~ 0
 GND
-Text Label 30900 17075 0    60   ~ 0
+Text Label 19375 15775 0    60   ~ 0
 GSM_POWER_KEY
 Text Label 22475 14325 0    60   ~ 0
@@
 Text Label 21350 14525 2    60   ~ 0
 XMEGA_PD0_GSM_POWER
-Text Label 29200 17825 2    60   ~ 0
+Text Label 17675 16525 2    60   ~ 0
 SIM_DET
-Text Label 29200 17900 2    60   ~ 0
+Text Label 17675 16600 2    60   ~ 0
 SIM_DATA
-Text Label 29200 17975 2    60   ~ 0
+Text Label 17675 16675 2    60   ~ 0
 SIM_CLK
-Text Label 29200 18050 2    60   ~ 0
+Text Label 17675 16750 2    60   ~ 0
 SIM_RST
-Text Label 29200 18125 2    60   ~ 0
+Text Label 17675 16825 2    60   ~ 0
 SIM_VDD
-NoConn ~ 30900 17150
-Text Label 30900 17600 0    60   ~ 0
+NoConn ~ 19375 15850
+Text Label 19375 16300 0    60   ~ 0
 GSM_ANT
 Text Label 22700 8550 2    60   ~ 0
 GSM_ANT
-Text Label 29200 17450 2    60   ~ 0
+Text Label 17675 16150 2    60   ~ 0
 GSM_MICP
-Text Label 29200 17525 2    60   ~ 0
+Text Label 17675 16225 2    60   ~ 0
 GSM_MICN
-Text Label 29200 17600 2    60   ~ 0
+Text Label 17675 16300 2    60   ~ 0
 GSM_SPKP
-Text Label 29200 17675 2    60   ~ 0
+Text Label 17675 16375 2    60   ~ 0
 GSM_SPKN
 $Sheet
@@
 	1    0    0    -1
 $EndComp
-NoConn ~ 30900 16850
-Text Label 30900 17300 0    60   ~ 0
-GND
-NoConn ~ 30900 17825
-NoConn ~ 30900 17900
-NoConn ~ 30900 18275
-NoConn ~ 30900 18350
-NoConn ~ 29200 18275
+NoConn ~ 19375 15550
+Text Label 19375 16000 0    60   ~ 0
+GND
+NoConn ~ 19375 16525
+NoConn ~ 19375 16600
+NoConn ~ 19375 16975
+NoConn ~ 19375 17050
+NoConn ~ 17675 16975
 Text Label 22525 17100 0    60   ~ 0
 SIM_DET
@@
 Text Label 22525 16900 0    60   ~ 0
 GND
-Text Label 30900 17000 0    60   ~ 0
+Text Label 19375 15700 0    60   ~ 0
 SIM_HOLDER_VDD_EXT
 Text Label 22525 17000 0    60   ~ 0
@@
 A7
 Wire Wire Line
-	33425 14800 33650 14800
+	33425 14800 33500 14800
+Wire Wire Line
+	33500 14800 33650 14800
 Wire Wire Line
 	34150 14800 34275 14800
@@
 Connection ~ 33500 14800
 Wire Wire Line
-	33350 14225 33650 14225
+	33350 14225 33500 14225
+Wire Wire Line
+	33500 14225 33650 14225
 Wire Wire Line
 	33550 14450 33500 14450
@@
 Connection ~ 33500 14225
 Wire Wire Line
-	33375 15375 33650 15375
+	33375 15375 33500 15375
+Wire Wire Line
+	33500 15375 33650 15375
 Wire Wire Line
 	33575 15625 33500 15625
@@
 	21250 11700 21250 12325
 Wire Wire Line
-	21000 11700 21875 11700
+	21000 11700 21250 11700
+Wire Wire Line
+	21250 11700 21875 11700
 Wire Wire Line
 	22750 12425 23025 12425
@@
 Connection ~ 21250 11700
 Wire Wire Line
-	24950 15950 25050 15950
+	24950 15950 25000 15950
+Wire Wire Line
+	25000 15950 25050 15950
 Wire Wire Line
 	25000 15950 25000 16025
@@
 	25350 15150 25350 15050
 Wire Wire Line
-	25000 16575 25425 16575
+	25000 16575 25350 16575
+Wire Wire Line
+	25350 16575 25425 16575
 Wire Wire Line
 	25000 16575 25000 16525
 Connection ~ 25350 16575
 Wire Wire Line
-	22475 14725 22475 15100
+	22475 14725 22475 14925
+Wire Wire Line
+	22475 14925 22475 15100
 Connection ~ 22475 14925
 Wire Wire Line
-	21850 14525 22175 14525
+	21850 14525 21975 14525
+Wire Wire Line
+	21975 14525 22175 14525
 Wire Wire Line
 	21975 14925 21975 14525
 Connection ~ 21975 14525
 Wire Wire Line
-	9775 10100 9300 10100
-Wire Wire Line
-	9550 9950 9550 10525
+	9775 10100 9550 10100
+Wire Wire Line
+	9550 10100 9300 10100
+Wire Wire Line
+	9550 9950 9550 10100
+Wire Wire Line
+	9550 10100 9550 10525
 Connection ~ 9550 10100
 Wire Wire Line
@@
 Connection ~ 28700 9575
 Wire Wire Line
-	28600 9250 28600 9750
+	28600 9250 28600 9575
+Wire Wire Line
+	28600 9575 28600 9750
 Connection ~ 28600 9575
 Wire Wire Line
@@
 	27050 14250 27400 14250
 Wire Wire Line
-	27600 9575 29300 9575
+	27600 9575 28100 9575
+Wire Wire Line
+	28100 9575 28200 9575
+Wire Wire Line
+	28200 9575 28225 9575
+Wire Wire Line
+	28225 9575 28300 9575
+Wire Wire Line
+	28300 9575 28350 9575
+Wire Wire Line
+	28350 9575 28400 9575
+Wire Wire Line
+	28400 9575 28475 9575
+Wire Wire Line
+	28475 9575 28500 9575
+Wire Wire Line
+	28500 9575 28600 9575
+Wire Wire Line
+	28600 9575 28700 9575
+Wire Wire Line
+	28700 9575 28725 9575
+Wire Wire Line
+	28725 9575 28800 9575
+Wire Wire Line
+	28800 9575 28850 9575
+Wire Wire Line
+	28850 9575 28900 9575
+Wire Wire Line
+	28900 9575 28975 9575
+Wire Wire Line
+	28975 9575 29300 9575
 Wire Wire Line
 	29300 9575 29300 9525
@@
 	29150 9750 29150 9675
 Wire Wire Line
-	30625 8925 30625 9975
+	30625 8925 30625 9000
+Wire Wire Line
+	30625 9000 30625 9300
+Wire Wire Line
+	30625 9300 30625 9675
+Wire Wire Line
+	30625 9675 30625 9975
 Wire Wire Line
 	29050 9625 30100 9625

Commit message: Design and connect GSM module.
Parts:
- removed D1: LED, LEDs:LED_0603, symbol LED-RESCUE-xmobile
- removed Q1, Q2: A2SHB, TO_SOT_Packages_SMD:SOT-23, symbol BC850
- removed R1, R2, R3, R4: 4.7KOmh, Resistors_SMD:R_0603_HandSoldering, symbol R-RESCUE-xmobile
- removed R10, R11, R12: 14KOmh, Resistors_SMD:R_0603_HandSoldering, symbol R-RESCUE-xmobile
- removed R13, R14, R15, R16, R7, R8, R9: 1KOmh, Resistors_SMD:R_0603_HandSoldering, symbol R-RESCUE-xmobile
- removed R5: 470Ом, Resistors_SMD:R_0603_HandSoldering, symbol R-RESCUE-xmobile
- removed U2: SIM800C, SIM800C_lup:SIM800C, symbol SIM800C
Connections:
- net labels added: GSM_CTS, GSM_DCD, GSM_DTR, GSM_PWRKEY, GSM_RI, GSM_RTS, GSM_RXD, GSM_TXD
- net labels removed: GSM_AT_CTS, GSM_AT_DCD, GSM_AT_DTR, GSM_AT_RI, GSM_AT_RTS, GSM_AT_RXD, GSM_AT_TXD, GSM_MICN, GSM_MICP, GSM_NETLIGHT, GSM_POWER_KEY, GSM_SPKN, GSM_SPKP, SIM_CLK, SIM_DATA, SIM_DET, SIM_HOLDER_VDD_EXT, SIM_RST, SIM_VDD
- wire segments 106 -> 60
- no-connect marks 60 -> 53
Other:
- moved on the sheet: C1, U1

Commit message: + new kbd, but not completed + SRAM lines(labels) replaced by bus
Parts:
- removed C1: C, Capacitors_SMD:C_1206_HandSoldering, symbol C-RESCUE-xmobile
- removed P1: USB_B, usb:Conn_USBmicro-B_ebay-side_TH, symbol USB_B
- removed P2: CONN_01X02, Connectors_JAE:JAE_LY20-04P-2T_2x02x2.00mm_Straight, symbol CONN_01X02
- removed U1: STF202-22T1G, semiconductor:TSOP-6, symbol STF202-22T1G
Connections:
- net labels added: ADDR_SRAM, DATA_SRAM
- net labels removed: 3.7V, GSM_ANT, GSM_USB_DN, GSM_USB_DP, GSM_USB_VBUS
- wire segments 60 -> 106
- no-connect marks 53 -> 52

Commit message: Added microSD slot.
Parts:
- added C?: C, 0.1u, symbol C
- added C?: CP, 10-100u, symbol CP
- added J?: TP_DISP_DATA_OUT, symbol TEST_1P
- added J?: Micro_SD_Card, microSD:microSD-noname, symbol Micro_SD_Card
Connections:
- net 3.3V: now also C?.1, C?.1, J?.4 (VDD)
- net EPD_BUSY: now also U?.J2 (PA3)
- net EPD_CLK: now also U?.H7 (PC5/XCK1/MOSI)
- net EPD_CS: now also U?.J7 (PC4/SS)
- net EPD_DC: now also U?.G2 (PA1)
- net EPD_DIN: now also U?.J8 (PC7/TXD1/SCK)
- net EPD_RST: now also U?.G3 (PA4)
- net GND: now also C?.2, C?.2, J?.6 (VSS)
- net microSD_CS: now reaches U?.F8 (PE1/XCK0/SCL)
- net microSD_CS: now also J?.2 (DAT3/CD)
- net KBD_SCL: now reaches U?.G6 (PC1/XCK0/SCL)
- net at U?.G7 (PC6/RXD1/MISO): now also J?.1
- net microSD_SCLK: now reaches U?.G8 (PD7/TXD1/SCK)
- net microSD_SCLK: now also J?.5 (CLK)
- net microSD_DO: now reaches U?.G9 (PD6/RXD1/MISO)
- net microSD_DO: now also J?.7 (DAT0)
- net GSM_STATUS: now reaches U?.H2 (PA2)
- net KBD_SDA: now reaches U?.H6 (PC0/SDA)
- net microSD_DI: now reaches U?.H8 (PD5/SCK1/MOSI)
- net microSD_DI: now also J?.3 (CMD)
- net KBD_INT: now reaches U?.J1 (PA0)
- no-connect marks 52 -> 55
Other:
- moved on the sheet: P3
Changed lines of the file:
@@
 L CONN_8 P3
 U 1 1 5974D7B3
-P 15400 1275
-F 0 "P3" V 15350 1275 60  0000 C CNN
-F 1 "CONN_8" V 15450 1275 60  0000 C CNN
-F 2 "Connectors_JAE:JAE_LY20-08P-2T_2x04x2.00mm_Straight" H 15400 1275 60  0001 C CNN
-F 3 "" H 15400 1275 60  0001 C CNN
-F 4 "EPD display connector" V 15575 1275 60  0000 C CNN "description"
-	1    15400 1275
-	1    0    0    -1
-$EndComp
-Text Label 15050 925  2    60   ~ 0
+P 13525 7500
+F 0 "P3" V 13475 7500 60  0000 C CNN
+F 1 "CONN_8" V 13575 7500 60  0000 C CNN
+F 2 "Connectors_JAE:JAE_LY20-08P-2T_2x04x2.00mm_Straight" H 13525 7500 60  0001 C CNN
+F 3 "" H 13525 7500 60  0001 C CNN
+F 4 "EPD display connector" V 13700 7500 60  0000 C CNN "description"
+	1    13525 7500
+	1    0    0    -1
+$EndComp
+Text Label 13175 7150 2    60   ~ 0
 EPD_BUSY
-Text Label 15050 1025 2    60   ~ 0
+Text Label 13175 7250 2    60   ~ 0
 EPD_RST
-Text Label 15050 1125 2    60   ~ 0
+Text Label 13175 7350 2    60   ~ 0
 EPD_DC
-Text Label 15050 1225 2    60   ~ 0
+Text Label 13175 7450 2    60   ~ 0
 EPD_CS
-Text Label 15050 1325 2    60   ~ 0
+Text Label 13175 7550 2    60   ~ 0
 EPD_CLK
-Text Label 15050 1425 2    60   ~ 0
+Text Label 13175 7650 2    60   ~ 0
 EPD_DIN
-Text Label 15050 1525 2    60   ~ 0
-GND
-Text Label 15050 1625 2    60   ~ 0
+Text Label 13175 7750 2    60   ~ 0
+GND
+Text Label 13175 7850 2    60   ~ 0
 3.3V
 Text Label 29800 12150 0    60   ~ 0
@@
 $EndSheet
 $Sheet
-S 550  10925 500  150
+S 14400 9675 500  150
 U 5A9FCB78
 F0 "xmega_power" 60
@@
 GND
 $Sheet
-S 13175 6900 650  675
+S 13125 6125 525  400
 U 5AA512DD
 F0 "xmobile_keyboard" 60
 F1 "xmobile_keyboard.sch" 60
-F2 "in1" I L 13175 7050 60
-F3 "in2" I L 13175 7200 60
-F4 "in3" I L 13175 7350 60
-F5 "out1" O R 13825 7050 60
-F6 "out2" O R 13825 7200 60
-F7 "out3" O R 13825 7350 60
-F8 "GND" B R 13825 7475 60
+F2 "SDA" B L 13125 6200 60
+F3 "SCL" B L 13125 6300 60
+F4 "INT" O L 13125 6400 60
 $EndSheet
-Text Label 13175 7050 2    60   ~ 0
-KBD_IN_1
 Text Label 29800 13100 0    60   ~ 0
 KBD_IN_1
 Text Label 29800 13200 0    60   ~ 0
 KBD_IN_2
-Text Label 13175 7200 2    60   ~ 0
-KBD_IN_2
 Text Label 29800 13300 0    60   ~ 0
-KBD_IN_3
-Text Label 13175 7350 2    60   ~ 0
 KBD_IN_3
 Text Label 29800 11750 0    60   ~ 0
 KBD_OUT_1
-Text Label 13825 7050 0    60   ~ 0
-KBD_OUT_1
 Text Label 29800 11850 0    60   ~ 0
 KBD_OUT_2
-Text Label 13825 7200 0    60   ~ 0
-KBD_OUT_2
 Text Label 29800 11950 0    60   ~ 0
-KBD_OUT_3
-Text Label 13825 7350 0    60   ~ 0
 KBD_OUT_3
 Text Label 29800 12600 0    60   ~ 0
@@
 NoConn ~ 8600 10100
 NoConn ~ 9300 9900
-Text Label 13825 7475 0    60   ~ 0
-GND
 NoConn ~ 34200 11550
 NoConn ~ 9650 10775
@@
 Text Label 3400 5450 2    60   ~ 0
 D0
-Text GLabel 825  10675 0    60   Input ~ 0
+Text GLabel 14675 9425 0    60   Input ~ 0
 3.3V
-Text Label 825  10675 0    60   ~ 0
+Text Label 14675 9425 0    60   ~ 0
 3.3V
 Wire Wire Line
@@
 Text Label 9500 3100 0    60   ~ 0
 3.3V
+Text Label 10800 6600 0    60   ~ 0
+EPD_RST
+Text Label 10800 6700 0    60   ~ 0
+EPD_BUSY
+Text Label 10800 6900 0    60   ~ 0
+EPD_DC
+Text Label 10800 4800 0    60   ~ 0
+EPD_CS
+Text Label 10800 4700 0    60   ~ 0
+EPD_CLK
+Text Label 10800 4500 0    60   ~ 0
+EPD_DIN
+Text Label 13125 6200 2    60   ~ 0
+KBD_SDA
+Text Label 13125 6300 2    60   ~ 0
+KBD_SCL
+Text Label 13125 6400 2    60   ~ 0
+KBD_INT
+Text Label 10800 5100 0    60   ~ 0
+KBD_SCL
+Text Label 10800 5200 0    60   ~ 0
+KBD_SDA
+Text Label 10800 7000 0    60   ~ 0
+KBD_INT
+$Comp
+L TEST_1P J?
+U 1 1 5C4B9CCC
+P 11625 4600
+F 0 "J?" H 11625 4870 50  0000 C CNN
+F 1 "TP_DISP_DATA_OUT" H 11625 4800 50  0000 C CNN
+F 2 "" H 11825 4600 50  0001 C CNN
+F 3 "" H 11825 4600 50  0001 C CNN
+	1    11625 4600
+	0    1    1    0
+$EndComp
+Wire Wire Line
+	10800 4600 11625 4600
+Text GLabel 15225 9425 0    60   Input ~ 0
+GND
+Text Label 15225 9425 0    60   ~ 0
+GND
+Text Label 12875 3550 0    60   ~ 0
+GSM_STATUS
+Text Label 10800 6800 0    60   ~ 0
+GSM_STATUS
+$Comp
+L Micro_SD_Card J?
+U 1 1 5C4DB2CD
+P 4075 8950
+F 0 "J?" H 3425 9550 50  0000 C CNN
+F 1 "Micro_SD_Card" H 4725 9550 50  0000 R CNN
+F 2 "microSD:microSD-noname" H 5225 9250 50  0001 C CNN
+F 3 "" H 4075 8950 50  0001 C CNN
+	1    4075 8950
+	1    0    0    -1
+$EndComp
+Text Label 3175 9150 2    60   ~ 0
+GND
+Text Label 3175 9050 2    60   ~ 0
+microSD_SCLK
+Text Label 1650 8950 2    60   ~ 0
+3.3V
+Text Label 3175 9250 2    60   ~ 0
+microSD_DO
+Text Label 3175 8750 2    60   ~ 0
+microSD_CS
+Text Label 3175 8850 2    60   ~ 0
+microSD_DI
+NoConn ~ 3175 8650
+NoConn ~ 3175 9350
+Text Label 1825 9525 3    60   ~ 0
+GND
+$Comp
+L C C?
+U 1 1 5C4DFD85
+P 1975 9100
+F 0 "C?" H 2000 9200 50  0000 L CNN
+F 1 "C" H 2000 9000 50  0000 L CNN
+F 2 "0.1u" H 2150 9075 50  0000 C CNN
+F 3 "" H 1975 9100 50  0001 C CNN
+	1    1975 9100
+	1    0    0    -1
+$EndComp
+$Comp
+L CP C?
+U 1 1 5C4DFEA4
+P 1650 9100
+F 0 "C?" H 1675 9200 50  0000 L CNN
+F 1 "CP" H 1675 9000 50  0000 L CNN
+F 2 "10-100u" H 1475 9000 50  0000 C CNN
+F 3 "" H 1650 9100 50  0001 C CNN
+	1    1650 9100
+	1    0    0    -1
+$EndComp
+Wire Wire Line
+	1650 8950 3175 8950
+Wire Wire Line
+	1650 9250 1975 9250
+Wire Wire Line
+	1825 9525 1825 9250
+Connection ~ 1825 9250
+Connection ~ 1975 8950
+NoConn ~ 4875 9550
+Text Label 10800 4100 0    60   ~ 0
+microSD_DI
+Text Label 10800 4300 0    60   ~ 0
+microSD_SCLK
+Text Label 10800 4200 0    60   ~ 0
+microSD_DO
+Text Label 10800 8000 0    60   ~ 0
+microSD_CS
 $EndSCHEMATC

Commit message: Add xmega pcb, Add SIM800 pcb Add SRAM pcb, Start to draw sim card holder pcb
Parts:
- U?: footprint (none) -> druid:48-ball_VFBGA_6x8x1mm_BV48BZ48
- U?: footprint (none) -> druid:BGA100_9x9x1.2_pitch-0.80mm
Changed lines of the file:
@@
 F 0 "U?" H 4250 5000 60  0000 C CNN
 F 1 "CY62158EV30LL-45BVXI" H 4250 5150 39  0000 C CNN
-F 2 "" H 4300 4250 60  0000 C CNN
+F 2 "druid:48-ball_VFBGA_6x8x1mm_BV48BZ48" H 4475 3925 60  0000 C CNN
 F 3 "" H 4300 4250 60  0000 C CNN
 	1    4250 5200
@@
 F 0 "U?" H 9300 4450 60  0000 C CNN
 F 1 "XMega128A1U_BGA100" H 9350 4900 60  0000 C CNN
-F 2 "" H 9700 7400 60  0000 C CNN
+F 2 "druid:BGA100_9x9x1.2_pitch-0.80mm" H 9400 5150 60  0000 C CNN
 F 3 "" H 9700 7400 60  0000 C CNN
 	1    9300 5600

Commit message: Old buttons replaced by membran buttons (electic and pcb) Added pcb for MAX7370 Cleared PCBs of resistor, capacitors and diodes
Parts:
- removed C2, C3, C32, C33, C34, C35, C36, C37, C38, C39: 100nF, Capacitors_SMD:C_0603_HandSoldering, symbol C
- removed C40, C41: 10mk, Capacitors_SMD:c_elec_4x5.3, symbol CP1-RESCUE-xmobile
- removed IC1: ATXMEGA128A1U-A, tqfp:LQFP-100_14x14mm_Pitch0.5mm, symbol ATXMEGA128A1U-A
- removed L1: 120m, Inductors:Inductor_1212, symbol INDUCTOR
- removed P10: CONN_01X08, Connectors_JAE:JAE_LY20-08P-2T_2x04x2.00mm_Straight, symbol CONN_01X08
- removed P7: CONN_4, Connectors_JAE:JAE_LY20-04P-2T_2x02x2.00mm_Straight, symbol CONN_4
- removed U5: switch1, switch1:switch_6x9, symbol switch1
- added SW?: SW_PUSH, druid:button_4pin_7,5x5, symbol SW_PUSH
- C?: value C -> 0.1u; footprint 0.1u -> (none)
- C?: value CP -> 10-100u; footprint 10-100u -> (none)
- R6: footprint Resistors_SMD:R_0603_HandSoldering -> (none)
Connections:
- net GND: now also SW?.1
- net PDI_C: now also SW?.2
- no-connect marks 55 -> 5

Commit message: Change PDI connector.
Parts:
- removed CON1: AVR-PDI-6, Connectors_JAE:JAE_LY20-06P-2T_2x03x2.00mm_Straight, symbol AVR-PDI-6
- added J?: Conn_01x04, symbol Conn_01x04
Connections:
- net 3.3V: now also J?.2 (Pin_2)
- net GND: now also J?.4 (Pin_4)
- net PDI_C: now also J?.3 (Pin_3)
- net PDI_D: now also J?.1 (Pin_1)
- no-connect marks 5 -> 3
Changed lines of the file:
@@
 F1 "xmega_power.sch" 60
 $EndSheet
-$Comp
-L AVR-PDI-6 CON1
-U 1 1 5AA047A2
-P 9650 10650
-F 0 "CON1" H 9570 10890 50  0000 C CNN
-F 1 "AVR-PDI-6" H 9440 10405 50  0000 L BNN
-F 2 "Connectors_JAE:JAE_LY20-06P-2T_2x03x2.00mm_Straight" V 10100 10700 50  0000 C CNN
-F 3 "" H 9650 10650 60  0001 C CNN
-	1    9650 10650
-	0    1    1    0
-$EndComp
-Text Label 9750 10775 3    60   ~ 0
+Text Label 9650 10700 1    60   ~ 0
 3.3V
-Text Label 9550 10775 3    60   ~ 0
+Text Label 9450 10700 1    60   ~ 0
 GND
 Text Label 8700 10100 2    60   ~ 0
@@
 F4 "INT" O L 13125 6400 60
 $EndSheet
-NoConn ~ 9650 10775
-NoConn ~ 9650 10525
 Text Label 9975 10325 0    60   ~ 0
 PDI_D
@@
 	9300 10100 9775 10100
 Wire Wire Line
-	9550 9950 9550 10525
+	9550 9950 9550 10700
 Connection ~ 9550 10100
 Wire Wire Line
-	9750 10525 9750 10325
+	9750 10325 9750 10700
 Wire Wire Line
 	9750 10325 9975 10325
@@
 F 0 "J?" H 3425 9550 50  0000 C CNN
 F 1 "Micro_SD_Card" H 4725 9550 50  0000 R CNN
-F 2 "microSD:microSD-noname" H 5225 9250 50  0001 C CNN
+F 2 "microSD:microSD-noname" H 4075 8200 50  0000 C CNN
 F 3 "" H 4075 8950 50  0001 C CNN
 	1    4075 8950
@@
 	1    0    0    -1
 $EndComp
+$Comp
+L Conn_01x04 J?
+U 1 1 5C50A6E4
+P 9650 10900
+F 0 "J?" H 9650 11100 50  0000 C CNN
+F 1 "Conn_01x04" V 9750 10850 50  0000 C CNN
+F 2 "" H 9650 10900 50  0001 C CNN
+F 3 "" H 9650 10900 50  0001 C CNN
+	1    9650 10900
+	0    1    1    0
+$EndComp
 $EndSCHEMATC
