File: druid/_autosave-xmobile.kicad_pcb (KiCad board)
At the start: 4 copper layers, 41.9 x 61.8 mm, 143 parts, among them J1 Micro_SD_Card, J2 TEST_VIBRO, J3 TEST_DISP_DATA_OUT, J4 USB_B_Micro, P1 CONN_8, Q1 BC850, Q2 BC850, SW1 SW_PUSH, SW10 SW_PUSH, SW11 SW_PUSH, SW12 SW_PUSH, SW13 SW_PUSH, SW14 SW_PUSH, SW15 SW_PUSH, SW16 SW_PUSH, SW17 SW_PUSH, SW18 SW_PUSH, SW19 SW_PUSH, SW2 SW_PUSH, SW20 SW_PUSH, SW21 SW_PUSH, SW3 SW_PUSH, SW4 SW_PUSH, SW5 SW_PUSH, SW6 SW_PUSH, SW7 SW_PUSH, SW8 SW_PUSH, SW9 SW_PUSH, U1 CY62158EV30LL-45BVXI, U2 XMega128A1U_BGA100, U3 TP4056, U4 TP4056, U5 XC6206P332MR, U6 MAX7370, U7 78646-3001, U8 SIM800C, U9 STF202-22T1G

Commit message: place components in rectangle.
Parts:
- moved C26 9.14 mm to (174.1, 127.9), turned to 180 degrees
- moved R6 6.23 mm to (177.1, 128.0), turned to 180 degrees
Changed lines of the file:
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@@
   (page A4)
   (layers
-    (0 F.Cu signal)
+    (0 F.Cu signal hide)
     (1 In1.Cu signal hide)
     (2 In2.Cu signal hide)
@@
     (34 B.Paste user hide)
     (35 F.Paste user hide)
-    (36 B.SilkS user hide)
+    (36 B.SilkS user)
     (37 F.SilkS user hide)
     (38 B.Mask user hide)
@@
   )
   (module Capacitor_SMD:C_0402_1005Metric (layer B.Cu)
-    (at 182.246265 123.718603)
+    (at 174.117 127.889 180)
     (descr "Capacitor SMD 0402 (1005 Metric), square (rectangular) end terminal, IPC_7351 nominal, (Body size source: http://www.tortai-tech.com/upload/download/2011102023233369053.pdf), generated with kicad-footprint-generator")
     (tags capacitor)
     (attr smd)
-    (fp_text reference C26 (at 0 1.17) (layer B.SilkS)
+    (fp_text reference C26 (at 0 1.17 180) (layer B.SilkS)
       (effects (font (size 0.5 0.5) (thickness 0.125)) (justify mirror))
     )
-    (fp_text value 10u (at 0 -1.17) (layer B.Fab)
+    (fp_text value 10u (at 0 -1.17 180) (layer B.Fab)
       (effects (font (size 0.5 0.5) (thickness 0.125)) (justify mirror))
     )
-    (fp_text user %R (at 0 0) (layer B.Fab)
+    (fp_text user %R (at 0 0 180) (layer B.Fab)
       (effects (font (size 0.25 0.25) (thickness 0.04)) (justify mirror))
     )
@@
     (fp_line (start -0.5 0.25) (end 0.5 0.25) (layer B.Fab) (width 0.1))
     (fp_line (start -0.5 -0.25) (end -0.5 0.25) (layer B.Fab) (width 0.1))
-    (pad 2 smd roundrect (at 0.485 0) (size 0.59 0.64) (layers B.Cu B.Paste B.Mask) (roundrect_rratio 0.25)
+    (pad 2 smd roundrect (at 0.485 0 180) (size 0.59 0.64) (layers B.Cu B.Paste B.Mask) (roundrect_rratio 0.25)
       (net 2 GND))
-    (pad 1 smd roundrect (at -0.485 0) (size 0.59 0.64) (layers B.Cu B.Paste B.Mask) (roundrect_rratio 0.25)
+    (pad 1 smd roundrect (at -0.485 0 180) (size 0.59 0.64) (layers B.Cu B.Paste B.Mask) (roundrect_rratio 0.25)
       (net 12 3.7V))
     (model ${KISYS3DMOD}/Capacitor_SMD.3dshapes/C_0402_1005Metric.wrl
@@
   )
   (module Resistor_SMD:R_0402_1005Metric (layer B.Cu)
-    (at 182.846265 125.698603)
+    (at 177.061 128.016 180)
     (descr "Resistor SMD 0402 (1005 Metric), square (rectangular) end terminal, IPC_7351 nominal, (Body size source: http://www.tortai-tech.com/upload/download/2011102023233369053.pdf), generated with kicad-footprint-generator")
     (tags resistor)
     (attr smd)
-    (fp_text reference R6 (at 0 1.17) (layer B.SilkS)
+    (fp_text reference R6 (at 0 1.17 180) (layer B.SilkS)
       (effects (font (size 0.5 0.5) (thickness 0.125)) (justify mirror))
     )
-    (fp_text value 1.2k (at 0 -1.17) (layer B.Fab)
+    (fp_text value 1.2k (at 0 -1.17 180) (layer B.Fab)
       (effects (font (size 0.5 0.5) (thickness 0.125)) (justify mirror))
     )
-    (fp_text user %R (at 0 0) (layer B.Fab)
+    (fp_text user %R (at 0 0 180) (layer B.Fab)
       (effects (font (size 0.25 0.25) (thickness 0.04)) (justify mirror))
     )
@@
     (fp_line (start -0.5 0.25) (end 0.5 0.25) (layer B.Fab) (width 0.1))
     (fp_line (start -0.5 -0.25) (end -0.5 0.25) (layer B.Fab) (width 0.1))
-    (pad 2 smd roundrect (at 0.485 0) (size 0.59 0.64) (layers B.Cu B.Paste B.Mask) (roundrect_rratio 0.25)
+    (pad 2 smd roundrect (at 0.485 0 180) (size 0.59 0.64) (layers B.Cu B.Paste B.Mask) (roundrect_rratio 0.25)
       (net 58 "Net-(R6-Pad2)"))
-    (pad 1 smd roundrect (at -0.485 0) (size 0.59 0.64) (layers B.Cu B.Paste B.Mask) (roundrect_rratio 0.25)
+    (pad 1 smd roundrect (at -0.485 0 180) (size 0.59 0.64) (layers B.Cu B.Paste B.Mask) (roundrect_rratio 0.25)
       (net 2 GND))
     (model ${KISYS3DMOD}/Resistor_SMD.3dshapes/R_0402_1005Metric.wrl
